Commit message: reformat URDF for readability

File: grippers/kinova_2f_lite/kinova_2f_lite_description/urdf/kinova_2f_lite_macro.urdf.xacro (robot description, xacro)
@@ -3,9 +3,13 @@
     <xacro:include filename="$(find kinova_2f_lite_description)/urdf/macros.urdf.xacro" />
     <xacro:property name="finger_to_control" value="right_finger_bottom_joint"/>
-    <xacro:macro name="load_gripper" params="*origin parent prefix sim_gazebo">
+    <xacro:macro name="load_gripper" params="
+        *origin
+        parent
+        prefix
+        sim_gazebo">
         <!-- Tool frame used by the arm -->
         <link name="${prefix}tool_frame"/>
         <joint name="${prefix}tool_frame_joint" type="fixed">
-            <origin xyz="0 0 0.130" rpy="0 0 1.57079632679" />
+            <origin rpy="0 0 1.57079632679" xyz="0 0 0.130" />
             <parent link="${prefix}${parent}" />
             <child link="${prefix}tool_frame" />
@@ -14,5 +18,5 @@
         <!-- Gripper description -->
         <joint name="${prefix}gripper_base_joint" type="fixed">
-            <origin xyz="0 0 0" rpy="0 0 0" />
+            <origin rpy="0 0 0" xyz="0 0 0" />
             <parent link="${prefix}${parent}" />
             <child link="${prefix}gripper_base_link" />
@@ -21,10 +25,13 @@
         <link name="${prefix}gripper_base_link">
             <inertial>
-                <origin xyz="4.03E-06 1.08E-05 0.041397" rpy="0 0 0" />
+                <origin rpy="0 0 0" xyz="4.03E-06 1.08E-05 0.041397" />
                 <mass value="0.1395" />
-                <inertia ixx="0.00011614" ixy="1E-08" ixz="4E-08" iyy="0.00010327" iyz="0" izz="9.707E-05" />
+                <inertia
+                    ixx="0.00011614" ixy="1E-08" ixz="4E-08"
+                    iyy="0.00010327" iyz="0"
+                    izz="9.707E-05" />
             </inertial>
             <visual>
-                <origin xyz="0 0 0" rpy="0 0 0" />
+                <origin rpy="0 0 0" xyz="0 0 0" />
                 <geometry>
                     <mesh filename="file://$(find kinova_2f_lite_description)/meshes/gripper_base_link.STL" />
@@ -35,5 +42,5 @@
             </visual>
             <collision>
-                <origin xyz="0 0 0" rpy="0 0 0" />
+                <origin rpy="0 0 0" xyz="0 0 0" />
                 <geometry>
                     <mesh filename="file://$(find kinova_2f_lite_description)/meshes/gripper_base_link.STL" />
@@ -43,10 +50,13 @@
         <link name="${prefix}right_finger_prox_link">
             <inertial>
-                <origin xyz="0.020257 0.0063483 6.991E-05" rpy="0 0 0" />
+                <origin rpy="0 0 0" xyz="0.020257 0.0063483 6.991E-05" />
                 <mass value="0.018385" />
-                <inertia ixx="2.29E-06" ixy="1.43E-06" ixz="0" iyy="4.56E-06" iyz="0" izz="4.77E-06" />
+                <inertia
+                    ixx="2.29E-06" ixy="1.43E-06" ixz="0"
+                    iyy="4.56E-06" iyz="0"
+                    izz="4.77E-06" />
             </inertial>
             <visual>
-                <origin xyz="0 0 0" rpy="0 0 0" />
+                <origin rpy="0 0 0" xyz="0 0 0" />
                 <geometry>
                     <mesh filename="file://$(find kinova_2f_lite_description)/meshes/right_finger_prox_link.STL" />
@@ -57,5 +67,5 @@
             </visual>
             <collision>
-                <origin xyz="0 0 0" rpy="0 0 0" />
+                <origin rpy="0 0 0" xyz="0 0 0" />
                 <geometry>
                     <mesh filename="file://$(find kinova_2f_lite_description)/meshes/right_finger_prox_link.STL" />
@@ -64,5 +74,5 @@
         </link>
         <joint name="${prefix}right_finger_bottom_joint" type="revolute">
-            <origin xyz="0 -0.030501 0.070003" rpy="0 1.5708 0" />
+            <origin rpy="0 1.5708 0" xyz="0 -0.030501 0.070003" />
             <parent link="${prefix}gripper_base_link" />
             <child link="${prefix}right_finger_prox_link" />
@@ -74,10 +84,13 @@
         <link name="${prefix}right_finger_dist_link">
             <inertial>
-                <origin xyz="0.018488 0.0011091 0" rpy="0 0 0" />
+                <origin rpy="0 0 0" xyz="0.018488 0.0011091 0" />
                 <mass value="0.010748" />
-                <inertia ixx="6.3E-07" ixy="3.2E-07" ixz="0" iyy="1.83E-06" iyz="0" izz="1.61E-06" />
+                <inertia
+                    ixx="6.3E-07" ixy="3.2E-07" ixz="0"
+                    iyy="1.83E-06" iyz="0"
+                    izz="1.61E-06" />
             </inertial>
             <visual>
-                <origin xyz="0 0 0" rpy="0 0 0" />
+                <origin rpy="0 0 0" xyz="0 0 0" />
                 <geometry>
                     <mesh filename="file://$(find kinova_2f_lite_description)/meshes/right_finger_dist_link.STL" />
@@ -88,5 +101,5 @@
             </visual>
             <collision>
-                <origin xyz="0 0 0" rpy="0 0 0" />
+                <origin rpy="0 0 0" xyz="0 0 0" />
                 <geometry>
                     <mesh filename="file://$(find kinova_2f_lite_description)/meshes/right_finger_dist_link.STL" />
@@ -96,5 +109,5 @@
         <joint name="${prefix}right_finger_tip_joint" type="revolute">
             <mimic joint="${prefix}right_finger_bottom_joint" multiplier="-1"/>
-            <origin xyz="-0.045636 0.020423 0" rpy="0 0 0" />
+            <origin rpy="0 0 0" xyz="-0.045636 0.020423 0" />
             <parent link="${prefix}right_finger_prox_link" />
             <child link="${prefix}right_finger_dist_link" />
@@ -106,10 +119,13 @@
         <link name="${prefix}left_finger_prox_link">
             <inertial>
-                <origin xyz="0.020257 0.0063483 6.99E-05" rpy="0 0 0" />
+                <origin rpy="0 0 0" xyz="0.020257 0.0063483 6.99E-05" />
                 <mass value="0.018385" />
-                <inertia ixx="2.29E-06" ixy="1.43E-06" ixz="0" iyy="4.56E-06" iyz="0" izz="4.77E-06" />
+                <inertia
+                    ixx="2.29E-06" ixy="1.43E-06" ixz="0"
+                    iyy="4.56E-06" iyz="0"
+                    izz="4.77E-06" />
             </inertial>
             <visual>
-                <origin xyz="0 0 0" rpy="0 0 0" />
+                <origin rpy="0 0 0" xyz="0 0 0" />
                 <geometry>
                     <mesh filename="file://$(find kinova_2f_lite_description)/meshes/left_finger_prox_link.STL" />
@@ -120,5 +136,5 @@
             </visual>
             <collision>
-                <origin xyz="0 0 0" rpy="0 0 0" />
+                <origin rpy="0 0 0" xyz="0 0 0" />
                 <geometry>
                     <mesh filename="file://$(find kinova_2f_lite_description)/meshes/left_finger_prox_link.STL" />
@@ -128,5 +144,5 @@
         <joint name="${prefix}left_finger_bottom_joint" type="revolute">
             <mimic joint="${prefix}right_finger_bottom_joint" multiplier="-1"/>
-            <origin xyz="0 0.0305 0.070003" rpy="0 1.5708 0" />
+            <origin rpy="0 1.5708 0" xyz="0 0.0305 0.070003" />
             <parent link="${prefix}gripper_base_link" />
             <child link="${prefix}left_finger_prox_link" />
@@ -138,10 +154,13 @@
         <link name="${prefix}left_finger_dist_link">
             <inertial>
-                <origin xyz="-0.018488 0.0011091 0" rpy="0 0 0" />
+                <origin rpy="0 0 0" xyz="-0.018488 0.0011091 0" />
                 <mass value="0.010748" />
-                <inertia ixx="6.3E-07" ixy="3.2E-07" ixz="0" iyy="1.83E-06" iyz="0" izz="1.61E-06" />
+                <inertia
+                    ixx="6.3E-07" ixy="3.2E-07" ixz="0"
+                    iyy="1.83E-06" iyz="0"
+                    izz="1.61E-06" />
             </inertial>
             <visual>
-                <origin xyz="0 0 0" rpy="0 0 0" />
+                <origin rpy="0 0 0" xyz="0 0 0" />
                 <geometry>
                     <mesh filename="file://$(find kinova_2f_lite_description)/meshes/left_finger_dist_link.STL" />
@@ -152,5 +171,5 @@
             </visual>
             <collision>
-                <origin xyz="0 0 0" rpy="0 0 0" />
+                <origin rpy="0 0 0" xyz="0 0 0" />
                 <geometry>
                     <mesh filename="file://$(find kinova_2f_lite_description)/meshes/left_finger_dist_link.STL" />
@@ -160,5 +179,5 @@
         <joint name="${prefix}left_finger_tip_joint" type="revolute">
             <mimic joint="${prefix}right_finger_bottom_joint" multiplier="-1"/>
-            <origin xyz="-0.045636 -0.020423 6.9901E-05" rpy="0 0 0" />
+            <origin rpy="0 0 0" xyz="-0.045636 -0.020423 6.9901E-05" />
             <parent link="${prefix}left_finger_prox_link" />
             <child link="${prefix}left_finger_dist_link" />
