Commit message: add ros2 control hardware interface for d1

File: grippers/d1_2f/d1_2f_description/urdf/d1_2f_macro.urdf.xacro (robot description, xacro)
@@ -3,7 +3,11 @@
     <xacro:include filename="$(find d1_2f_description)/urdf/macros.urdf.xacro" />
     <xacro:property name="finger_to_control" value="joint_R"/>
-    <xacro:macro name="load_gripper" params="*origin parent prefix sim_gazebo">
+    <xacro:macro name="load_gripper" params="
+        *origin
+        parent
+        prefix
+        sim_gazebo">
         <joint name="${prefix}gripper_base_joint" type="fixed">
-            <xacro:insert_block name="origin"/>
+            <xacro:insert_block name="origin" />
             <parent link="${prefix}${parent}" />
             <child link="${prefix}gripper_base_link" />
@@ -12,27 +16,30 @@
         <link name="${prefix}gripper_base_link">
             <inertial>
-                <origin xyz="-0.0068528 -3.9973E-06 0.039705" rpy="0 0 0"/>
-                <mass value="0.077892"/>
-                <inertia ixx="3.8236E-05" ixy="1.3465E-08" ixz="-2.0614E-07" iyy="1.7707E-05" iyz="-6.7117E-10" izz="4.8839E-05"/>
+                <origin rpy="0 0 0" xyz="-0.0068528 -3.9973E-06 0.039705" />
+                <mass value="0.077892" />
+                <inertia
+                    ixx="3.8236E-05" ixy="1.3465E-08" ixz="-2.0614E-07"
+                    iyy="1.7707E-05" iyz="-6.7117E-10"
+                    izz="4.8839E-05" />
             </inertial>
             <visual>
-                <origin xyz="0 0 0" rpy="0 0 0"/>
+                <origin rpy="0 0 0" xyz="0 0 0" />
                 <geometry>
-                    <mesh filename="file://$(find unitree_d1_description)/meshes/Link6.STL"/>
+                    <mesh filename="file://$(find unitree_d1_description)/meshes/Link6.STL" />
                 </geometry>
-                <xacro:insert_block name="material_black"/>
+                <xacro:insert_block name="material_black" />
             </visual>
             <collision>
-                <origin xyz="0 0 0" rpy="0 0 0"/>
+                <origin rpy="0 0 0" xyz="0 0 0" />
                 <geometry>
-                    <mesh filename="file://$(find unitree_d1_description)/meshes/Link6.STL"/>
+                    <mesh filename="file://$(find unitree_d1_description)/meshes/Link6.STL" />
                 </geometry>
             </collision>
         </link>
         <joint name="${prefix}joint_L" type="prismatic">
-            <origin xyz="-0.0056012 -0.029636 0.0706" rpy="-1.5714 -1.5708 0" />
+            <origin rpy="-1.5714 -1.5708 0" xyz="-0.0056012 -0.029636 0.0706" />
             <parent link="${prefix}gripper_base_link" />
             <child link="${prefix}Link_L" />
-            <axis xyz="0 0 -1"/>
+            <axis xyz="0 0 -1" />
             <limit lower="${min_left_finger_joint_pos}" upper="${max_left_finger_joint_pos}"
                     effort="${left_finger_joint_effort}" velocity="${left_finger_joint_vel}" />
@@ -41,61 +48,55 @@
         <link name="${prefix}Link_L">
             <inertial>
-                <origin xyz="0.018927 0.006 0.012082" rpy="0 0 0"/>
-                <mass value="0.015046"/>
+                <origin rpy="0 0 0" xyz="0.018927 0.006 0.012082" />
+                <mass value="0.015046" />
                 <inertia
-                    ixx="1.2692E-06"
-                    ixy="7.7441E-20"
-                    ixz="-1.133E-07"
-                    iyy="2.0229E-06"
-                    iyz="1.2044E-20"
+                    ixx="1.2692E-06" ixy="7.7441E-20" ixz="-1.133E-07"
+                    iyy="2.0229E-06" iyz="1.2044E-20"
                     izz="2.6177E-06" />
             </inertial>
             <visual>
-                <origin xyz="0 0 0" rpy="0 0 0"/>
+                <origin rpy="0 0 0" xyz="0 0 0" />
                 <geometry>
-                    <mesh filename="file://$(find d1_2f_description)/meshes/Link_L.STL"/>
+                    <mesh filename="file://$(find d1_2f_description)/meshes/Link_L.STL" />
                 </geometry>
-                <xacro:insert_block name="material_black"/>
+                <xacro:insert_block name="material_black" />
             </visual>
             <collision>
-                <origin xyz="0 0 0" rpy="0 0 0"/>
+                <origin rpy="0 0 0" xyz="0 0 0" />
                 <geometry>
-                    <mesh filename="file://$(find d1_2f_description)/meshes/Link_L.STL"/>
+                    <mesh filename="file://$(find d1_2f_description)/meshes/Link_L.STL" />
                 </geometry>
             </collision>
         </link>
         <joint name="${prefix}joint_R" type="prismatic">
-            <mimic joint="${prefix}joint_L" multiplier="-1"/>
-            <origin xyz="-0.0056388 0.02964 0.0706" rpy="1.5702 -1.5708 0"/>
-            <parent link="${prefix}gripper_base_link"/>
-            <child link="${prefix}link_R"/>
-            <axis xyz="0 0 1"/>
+            <mimic joint="${prefix}joint_L" multiplier="-1" />
+            <origin rpy="1.5702 -1.5708 0" xyz="-0.0056388 0.02964 0.0706" />
+            <parent link="${prefix}gripper_base_link" />
+            <child link="${prefix}Link_R" />
+            <axis xyz="0 0 1" />
             <limit lower="${min_right_finger_joint_pos}" upper="${max_right_finger_joint_pos}"
                     effort="${right_finger_joint_effort}" velocity="${right_finger_joint_vel}" />
             <dynamics damping="${right_finger_joint_damping}" friction="${right_finger_joint_friction}" />
         </joint>
-        <link name="${prefix}link_R">
+        <link name="${prefix}Link_R">
             <inertial>
-                <origin xyz="0.018927 -0.006 0.012082" rpy="0 0 0"/>
-                <mass value="0.015046"/>
+                <origin rpy="0 0 0" xyz="0.018927 -0.006 0.012082" />
+                <mass value="0.015046" />
                 <inertia
-                    ixx="1.2692E-06"
-                    ixy="-7.8273E-20"
-                    ixz="-1.133E-07"
-                    iyy="2.0229E-06"
-                    iyz="-1.2122E-20"
+                    ixx="1.2692E-06" ixy="-7.8273E-20" ixz="-1.133E-07"
+                    iyy="2.0229E-06" iyz="-1.2122E-20"
                     izz="2.6177E-06" />
             </inertial>
             <visual>
-                <origin xyz="0 0 0" rpy="0 0 0"/>
+                <origin rpy="0 0 0" xyz="0 0 0" />
                 <geometry>
-                    <mesh filename="file://$(find d1_2f_description)/meshes/Link_R.STL"/>
+                    <mesh filename="file://$(find d1_2f_description)/meshes/Link_R.STL" />
                 </geometry>
-                <xacro:insert_block name="material_black"/>
+                <xacro:insert_block name="material_black" />
             </visual>
             <collision>
-                <origin xyz="0 0 0" rpy="0 0 0"/>
+                <origin rpy="0 0 0" xyz="0 0 0" />
                 <geometry>
-                    <mesh filename="file://$(find d1_2f_description)/meshes/Link_R.STL"/>
+                    <mesh filename="file://$(find d1_2f_description)/meshes/Link_R.STL" />
                 </geometry>
             </collision>

File: unitree_d1/unitree_d1_description/urdf/ros2_control/unitree_d1_ros2_control.xacro (robot description, xacro)
@@ -8,4 +8,16 @@
             </hardware>
         </xacro:if>
+        <xacro:unless value="${sim_gazebo}">
+            <hardware>
+                <plugin>d1_hardware_interface/D1HardwareInterface</plugin>
+                <!-- <param name="topic_sufix">asda</param> -->
+                <!-- <xacro:if value="${gripper == 'z1_1f'}">
+                    <param name="gripper">true</param>
+                </xacro:if>
+                <xacro:unless value="${gripper == 'z1_1f'}">
+                    <param name="gripper">false</param>
+                </xacro:unless> -->
+            </hardware>
+        </xacro:unless>
         <joint name="${prefix}joint_1">
             <command_interface name="position">
@@ -13,9 +25,14 @@
                 <param name="max">${max_joint_1_pos}</param>
             </command_interface>
-            <state_interface name="position">
-                <param name="initial_value">${joint_1_initial}</param>
-            </state_interface>
-            <state_interface name="velocity"/>
-            <state_interface name="effort"/>
+            <xacro:if value="${sim_gazebo}">
+                <state_interface name="position">
+                    <param name="initial_value">${joint_1_initial}</param>
+                </state_interface>
+            </xacro:if>
+            <xacro:unless value="${sim_gazebo}">
+                <state_interface name="position" />
+            </xacro:unless>
+            <!-- <state_interface name="velocity"/>
+            <state_interface name="effort"/> -->
         </joint>
         <joint name="${prefix}joint_2">
@@ -24,9 +41,14 @@
                 <param name="max">${max_joint_2_pos}</param>
             </command_interface>
-            <state_interface name="position">
-                <param name="initial_value">${joint_2_initial}</param>
-            </state_interface>
-            <state_interface name="velocity"/>
-            <state_interface name="effort"/>
+            <xacro:if value="${sim_gazebo}">
+                <state_interface name="position">
+                    <param name="initial_value">${joint_2_initial}</param>
+                </state_interface>
+            </xacro:if>
+            <xacro:unless value="${sim_gazebo}">
+                <state_interface name="position" />
+            </xacro:unless>
+            <!-- <state_interface name="velocity"/>
+            <state_interface name="effort"/> -->
         </joint>
         <joint name="${prefix}joint_3">
@@ -35,9 +57,14 @@
                 <param name="max">${max_joint_3_pos}</param>
             </command_interface>
-            <state_interface name="position">
-                <param name="initial_value">${joint_3_initial}</param>
-            </state_interface>
-            <state_interface name="velocity"/>
-            <state_interface name="effort"/>
+            <xacro:if value="${sim_gazebo}">
+                <state_interface name="position">
+                    <param name="initial_value">${joint_3_initial}</param>
+                </state_interface>
+            </xacro:if>
+            <xacro:unless value="${sim_gazebo}">
+                <state_interface name="position" />
+            </xacro:unless>
+            <!-- <state_interface name="velocity"/>
+            <state_interface name="effort"/> -->
         </joint>
         <joint name="${prefix}joint_4">
@@ -46,9 +73,14 @@
                 <param name="max">${max_joint_4_pos}</param>
             </command_interface>
-            <state_interface name="position">
-                <param name="initial_value">${joint_4_initial}</param>
-            </state_interface>
-            <state_interface name="velocity"/>
-            <state_interface name="effort"/>
+            <xacro:if value="${sim_gazebo}">
+                <state_interface name="position">
+                    <param name="initial_value">${joint_4_initial}</param>
+                </state_interface>
+            </xacro:if>
+            <xacro:unless value="${sim_gazebo}">
+                <state_interface name="position" />
+            </xacro:unless>
+            <!-- <state_interface name="velocity"/>
+            <state_interface name="effort"/> -->
         </joint>
         <joint name="${prefix}joint_5">
@@ -57,9 +89,14 @@
                 <param name="max">${max_joint_5_pos}</param>
             </command_interface>
-            <state_interface name="position">
-                <param name="initial_value">${joint_5_initial}</param>
-            </state_interface>
-            <state_interface name="velocity"/>
-            <state_interface name="effort"/>
+            <xacro:if value="${sim_gazebo}">
+                <state_interface name="position">
+                    <param name="initial_value">${joint_5_initial}</param>
+                </state_interface>
+            </xacro:if>
+            <xacro:unless value="${sim_gazebo}">
+                <state_interface name="position" />
+            </xacro:unless>
+            <!-- <state_interface name="velocity"/>
+            <state_interface name="effort"/> -->
         </joint>
         <joint name="${prefix}joint_6">
@@ -68,9 +105,14 @@
                 <param name="max">${max_joint_6_pos}</param>
             </command_interface>
-            <state_interface name="position">
-                <param name="initial_value">${joint_6_initial}</param>
-            </state_interface>
-            <state_interface name="velocity"/>
-            <state_interface name="effort"/>
+            <xacro:if value="${sim_gazebo}">
+                <state_interface name="position">
+                    <param name="initial_value">${joint_6_initial}</param>
+                </state_interface>
+            </xacro:if>
+            <xacro:unless value="${sim_gazebo}">
+                <state_interface name="position" />
+            </xacro:unless>
+            <!-- <state_interface name="velocity"/>
+            <state_interface name="effort"/> -->
         </joint>
     </ros2_control>

File: unitree_d1/unitree_d1_description/urdf/unitree_d1.urdf.xacro (robot description, xacro)
@@ -1,8 +1,7 @@
 <?xml version="1.0"?>
-<robot name="$(arg name)" xmlns:xacro="http://ros.org/wiki/xacro">
+<robot name="unitree_d1" xmlns:xacro="http://ros.org/wiki/xacro">
     <!-- Arguments -->
     <xacro:arg name="sim_gazebo" default="true" />
-    <xacro:arg name="use_camera" default="true" />
-    <xacro:arg name="parent" default="world"/>
+    <xacro:arg name="use_camera" default="false" />
     <xacro:arg name="prefix" default=""/>
     <xacro:arg name="gripper" default="" />
@@ -12,18 +11,21 @@
     <xacro:include filename="$(find unitree_d1_description)/urdf/macros.urdf.xacro" />
     <link name="world"/>
-    <xacro:load_arm parent="$(arg parent)"
+    <xacro:load_arm
+        parent="world"
+        prefix="$(arg prefix)"
+        sim_gazebo="$(arg sim_gazebo)"
+        gripper="$(arg gripper)"
+        use_camera="$(arg use_camera)">
+        <origin rpy="0 0 0" xyz="0 0 0" />
+    </xacro:load_arm>
+    <xacro:property name="gripper_pkg" value="$(arg gripper)_description" />
+    <xacro:unless value="${not '$(arg gripper)'}">
+        <xacro:include filename="$(find ${gripper_pkg})/urdf/$(arg gripper)_macro.urdf.xacro" />
+        <xacro:load_gripper
+            parent="${last_arm_link}"
             prefix="$(arg prefix)"
-            sim_gazebo="$(arg sim_gazebo)"
-            gripper="$(arg gripper)"
-            use_camera="$(arg use_camera)" >
-        <origin xyz="0 0 0" rpy="0 0 0" />
-    </xacro:load_arm>
-    <xacro:unless value="${not '$(arg gripper)'}" >
-        <xacro:include filename="$(find d1_2f_description)/urdf/d1_2f_macro.urdf.xacro" />
-        <xacro:load_gripper parent="${last_arm_link}"
-                prefix="$(arg prefix)"
-                sim_gazebo="$(arg sim_gazebo)" >
-            <!-- <origin xyz="-0.0056012 -0.029636 0.0706" rpy="-1.5714 -1.5708 0" /> -->
-            <origin xyz="0.0 0.0 0.0" rpy="0.0 0.0 0.0" />
+            sim_gazebo="$(arg sim_gazebo)">
+            <!-- <origin rpy="-1.5714 -1.5708 0" xyz="-0.0056012 -0.029636 0.0706" /> -->
+            <origin rpy="0 0 0" xyz="0 0 0" />
         </xacro:load_gripper>
     </xacro:unless>
