Commit message: add ros2 control hardware interface for d1

File: unitree_d1/unitree_d1_description/urdf/unitree_d1_macro.urdf.xacro (robot description, xacro)
@@ -11,17 +11,20 @@
         <link name="${prefix}base_link">
             <inertial>
-                <origin xyz="-0.00048697 -2.9605E-12 0.017142" rpy="0 0 0"/>
-                <mass value="0.077233"/>
-                <inertia ixx="0.00010316" ixy="-1.0285E-14" ixz="2.0449E-07" iyy="0.00011888" iyz="7.3026E-15" izz="0.00018362"/>
-            </inertial>
-            <visual>
-                <origin xyz="0 0 0" rpy="0 0 0"/>
+                <origin rpy="0 0 0" xyz="-0.00048697 -2.9605E-12 0.017142" />
+                <mass value="0.077233" />
+                <inertia
+                    ixx="0.00010316" ixy="-1.0285E-14" ixz="2.0449E-07"
+                    iyy="0.00011888" iyz="7.3026E-15"
+                    izz="0.00018362" />
+            </inertial>
+            <visual>
+                <origin rpy="0 0 0" xyz="0 0 0" />
                 <geometry>
                     <mesh filename="file://$(find unitree_d1_description)/meshes/base_link.STL" />
                 </geometry>
-                <xacro:insert_block name="material_black"/>
-            </visual>
-            <collision>
-                <origin xyz="0 0 0" rpy="0 0 0"/>
+                <xacro:insert_block name="material_black" />
+            </visual>
+            <collision>
+                <origin rpy="0 0 0" xyz="0 0 0" />
                 <geometry>
                     <mesh filename="file://$(find unitree_d1_description)/meshes/base_link.STL" />
@@ -31,27 +34,30 @@
         <link name="${prefix}Link1">
             <inertial>
-                <origin xyz="0.0024649 0.00010517 0.032696" rpy="0 0 0"/>
-                <mass value="0.13174"/>
-                <inertia ixx="6.7236E-05" ixy="-5.5664E-08" ixz="7.0454E-08" iyy="5.416E-05" iyz="-3.5709E-07" izz="4.6637E-05"/>
-            </inertial>
-            <visual>
-                <origin xyz="0 0 0" rpy="0 0 0"/>
-                <geometry>
-                    <mesh filename="file://$(find unitree_d1_description)/meshes/Link1.STL"/>
-                </geometry>
-                <xacro:insert_block name="material_black"/>
-            </visual>
-            <collision>
-                <origin xyz="0 0 0" rpy="0 0 0"/>
-                <geometry>
-                    <mesh filename="file://$(find unitree_d1_description)/meshes/Link1.STL"/>
+                <origin rpy="0 0 0" xyz="0.0024649 0.00010517 0.032696" />
+                <mass value="0.13174" />
+                <inertia
+                    ixx="6.7236E-05" ixy="-5.5664E-08" ixz="7.0454E-08"
+                    iyy="5.416E-05" iyz="-3.5709E-07"
+                    izz="4.6637E-05" />
+            </inertial>
+            <visual>
+                <origin rpy="0 0 0" xyz="0 0 0" />
+                <geometry>
+                    <mesh filename="file://$(find unitree_d1_description)/meshes/Link1.STL" />
+                </geometry>
+                <xacro:insert_block name="material_black" />
+            </visual>
+            <collision>
+                <origin xyz="0 0 0" rpy="0 0 0" />
+                <geometry>
+                    <mesh filename="file://$(find unitree_d1_description)/meshes/Link1.STL" />
                 </geometry>
             </collision>
         </link>
         <joint name="${prefix}joint_1" type="revolute">
-            <origin xyz="0 0 0.0533" rpy="0 0 -3.1416"/>
-            <parent link="${prefix}base_link"/>
-            <child link="${prefix}Link1"/>
-            <axis xyz="0 0 1"/>
+            <origin rpy="0 0 -3.1416" xyz="0 0 0.0533" />
+            <parent link="${prefix}base_link" />
+            <child link="${prefix}Link1" />
+            <axis xyz="0 0 1" />
             <limit lower="${min_joint_1_pos}" upper="${max_joint_1_pos}"
                     effort="${joint_1_effort}" velocity="${joint_1_vel}" />
@@ -59,10 +65,13 @@
         <link name="${prefix}Link2">
             <inertial>
-                <origin xyz="0.0002018 0.19201 -0.027007" rpy="0 0 0"/>
-                <mass value="0.20213"/>
-                <inertia ixx="0.00025682" ixy="-1.139E-07" ixz="5.5667E-08" iyy="6.3307E-05" iyz="-3.5717E-07" izz="0.00022968"/>
-            </inertial>
-            <visual>
-                <origin xyz="0 0 0" rpy="0 0 0"/>
+                <origin rpy="0 0 0" xyz="0.0002018 0.19201 -0.027007" />
+                <mass value="0.20213" />
+                <inertia
+                    ixx="0.00025682" ixy="-1.139E-07" ixz="5.5667E-08"
+                    iyy="6.3307E-05" iyz="-3.5717E-07"
+                    izz="0.00022968" />
+            </inertial>
+            <visual>
+                <origin rpy="0 0 0" xyz="0 0 0" />
                 <geometry>
                     <mesh filename="file://$(find unitree_d1_description)/meshes/Link2.STL"/>
@@ -71,5 +80,5 @@
             </visual>
             <collision>
-                <origin xyz="0 0 0" rpy="0 0 0"/>
+                <origin rpy="0 0 0" xyz="0 0 0" />
                 <geometry>
                     <mesh filename="file://$(find unitree_d1_description)/meshes/Link2.STL"/>
@@ -78,8 +87,8 @@
         </link>
         <joint name="${prefix}joint_2" type="revolute">
-            <origin xyz="0 0.028 0.0563" rpy="1.5708 0 -3.1416"/>
-            <parent link="${prefix}Link1"/>
-            <child link="${prefix}Link2"/>
-            <axis xyz="0 0 -1"/>
+            <origin rpy="1.5708 0 -3.1416" xyz="0 0.028 0.0563" />
+            <parent link="${prefix}Link1" />
+            <child link="${prefix}Link2" />
+            <axis xyz="0 0 -1" />
             <limit lower="${min_joint_2_pos}" upper="${max_joint_2_pos}"
                     effort="${joint_2_effort}" velocity="${joint_2_vel}" />
@@ -87,27 +96,30 @@
         <link name="${prefix}Link3">
             <inertial>
-                <origin xyz="0.015164 0.044482 -0.027461" rpy="0 0 0"/>
-                <mass value="0.0629"/>
-                <inertia ixx="1.7232E-05" ixy="-2.6967E-06" ixz="-9.4911E-11" iyy="1.2606E-05" iyz="-9.9169E-11" izz="1.4964E-05"/>
-            </inertial>
-            <visual>
-                <origin xyz="0 0 0" rpy="0 0 0"/>
-                <geometry>
-                    <mesh filename="file://$(find unitree_d1_description)/meshes/Link3.STL"/>
-                </geometry>
-                <xacro:insert_block name="material_black"/>
-            </visual>
-            <collision>
-                <origin xyz="0 0 0" rpy="0 0 0"/>
-                <geometry>
-                    <mesh filename="file://$(find unitree_d1_description)/meshes/Link3.STL"/>
+                <origin rpy="0 0 0" xyz="0.015164 0.044482 -0.027461" />
+                <mass value="0.0629" />
+                <inertia
+                    ixx="1.7232E-05" ixy="-2.6967E-06" ixz="-9.4911E-11"
+                    iyy="1.2606E-05" iyz="-9.9169E-11"
+                    izz="1.4964E-05" />
+            </inertial>
+            <visual>
+                <origin rpy="0 0 0" xyz="0 0 0" />
+                <geometry>
+                    <mesh filename="file://$(find unitree_d1_description)/meshes/Link3.STL" />
+                </geometry>
+                <xacro:insert_block name="material_black" />
+            </visual>
+            <collision>
+                <origin rpy="0 0 0" xyz="0 0 0" />
+                <geometry>
+                    <mesh filename="file://$(find unitree_d1_description)/meshes/Link3.STL" />
                 </geometry>
             </collision>
         </link>
         <joint name="${prefix}joint_3" type="revolute">
-            <origin xyz="0 0.2693 0.0009" rpy="0 0 0"/>
-            <parent link="${prefix}Link2"/>
-            <child link="${prefix}Link3"/>
-            <axis xyz="0 0 -1"/>
+            <origin rpy="0 0 0" xyz="0 0.2693 0.0009" />
+            <parent link="${prefix}Link2" />
+            <child link="${prefix}Link3" />
+            <axis xyz="0 0 -1" />
             <limit lower="${min_joint_3_pos}" upper="${max_joint_3_pos}"
                     effort="${joint_3_effort}" velocity="${joint_3_vel}" />
@@ -115,24 +127,27 @@
         <link name="${prefix}Link4">
             <inertial>
-                <origin xyz="-0.00029556 -0.00016104 0.091339" rpy="0 0 0"/>
-                <mass value="0.083332"/>
-                <inertia ixx="3.9308E-05" ixy="1.0126E-08" ixz="-9.4316E-08" iyy="3.4378E-05" iyz="-1.6915E-09" izz="1.1597E-05"/>
-            </inertial>
-            <visual>
-                <origin xyz="0 0 0" rpy="0 0 0"/>
-                <geometry>
-                    <mesh filename="file://$(find unitree_d1_description)/meshes/Link4.STL"/>
-                </geometry>
-                <xacro:insert_block name="material_black"/>
-            </visual>
-            <collision>
-                <origin xyz="0 0 0" rpy="0 0 0"/>
-                <geometry>
-                    <mesh filename="file://$(find unitree_d1_description)/meshes/Link4.STL"/>
+                <origin rpy="0 0 0" xyz="-0.00029556 -0.00016104 0.091339" />
+                <mass value="0.083332" />
+                <inertia
+                    ixx="3.9308E-05" ixy="1.0126E-08" ixz="-9.4316E-08"
+                    iyy="3.4378E-05" iyz="-1.6915E-09"
+                    izz="1.1597E-05" />
+            </inertial>
+            <visual>
+                <origin rpy="0 0 0" xyz="0 0 0" />
+                <geometry>
+                    <mesh filename="file://$(find unitree_d1_description)/meshes/Link4.STL" />
+                </geometry>
+                <xacro:insert_block name="material_black" />
+            </visual>
+            <collision>
+                <origin rpy="0 0 0" xyz="0 0 0" />
+                <geometry>
+                    <mesh filename="file://$(find unitree_d1_description)/meshes/Link4.STL" />
                 </geometry>
             </collision>
         </link>
         <joint name="${prefix}joint_4" type="revolute">
-            <origin xyz="0.0577 0.042 -0.0275" rpy="-1.5708 0 -1.5708"/>
+            <origin rpy="-1.5708 0 -1.5708" xyz="0.0577 0.042 -0.0275" />
             <parent link="${prefix}Link3"/>
             <child link="${prefix}Link4"/>
@@ -143,55 +158,48 @@
         <link name="${prefix}Link5">
             <inertial>
-                <origin xyz="0.040573 0.0062891 -0.023838" rpy="0 0 0"/>
-                <mass value="0.053817"/>
-                <inertia ixx="1.3072E-05" ixy="-3.9511E-07" ixz="-3.1889E-10" iyy="8.6301E-06" iyz="-1.8416E-09" izz="1.1049E-05"/>
-            </inertial>
-            <visual>
-                <origin xyz="0 0 0" rpy="0 0 0"/>
-                <geometry>
-                    <mesh filename="file://$(find unitree_d1_description)/meshes/Link5.STL"/>
-                </geometry>
-                <xacro:insert_block name="material_black"/>
-            </visual>
-            <collision>
-                <origin xyz="0 0 0" rpy="0 0 0"/>
-                <geometry>
-                    <mesh filename="file://$(find unitree_d1_description)/meshes/Link5.STL"/>
+                <origin rpy="0 0 0" xyz="0.040573 0.0062891 -0.023838" />
+                <mass value="0.053817" />
+                <inertia
+                    ixx="1.3072E-05" ixy="-3.9511E-07" ixz="-3.1889E-10"
+                    iyy="8.6301E-06" iyz="-1.8416E-09"
+                    izz="1.1049E-05" />
+            </inertial>
+            <visual>
+                <origin xyz="0 0 0" rpy="0 0 0" />
+                <geometry>
+                    <mesh filename="file://$(find unitree_d1_description)/meshes/Link5.STL" />
+                </geometry>
+                <xacro:insert_block name="material_black" />
+            </visual>
+            <collision>
+                <origin rpy="0 0 0" xyz="0 0 0" />
+                <geometry>
+                    <mesh filename="file://$(find unitree_d1_description)/meshes/Link5.STL" />
                 </geometry>
             </collision>
         </link>
         <joint name="${prefix}joint_5" type="revolute">
-            <origin xyz="-0.0001 -0.0237 0.14018" rpy="1.5708 -1.5708 0"/>
-            <parent link="${prefix}Link4"/>
-            <child link="${prefix}Link5"/>
-            <axis xyz="0 0 -1"/>
+            <origin rpy="1.5708 -1.5708 0" xyz="-0.0001 -0.0237 0.14018" />
+            <parent link="${prefix}Link4" />
+            <child link="${prefix}Link5" />
+            <axis xyz="0 0 -1" />
             <limit lower="${min_joint_5_pos}" upper="${max_joint_5_pos}"
                     effort="${joint_5_effort}" velocity="${joint_5_vel}" />
         </joint>
         <link name="${prefix}Link6">
-            <!-- <inertial>
-                <origin xyz="-0.0068528 -3.9973E-06 0.039705" rpy="0 0 0"/>
-                <mass value="0.077892"/>
-                <inertia ixx="3.8236E-05" ixy="1.3465E-08" ixz="-2.0614E-07" iyy="1.7707E-05" iyz="-6.7117E-10" izz="4.8839E-05"/>
-            </inertial>
-            <visual>
-                <origin xyz="0 0 0" rpy="0 0 0"/>
-                <geometry>
-                    <mesh filename="file://$(find unitree_d1_description)/meshes/Link6.STL"/>
-                </geometry>
-                <xacro:insert_block name="material_dark_grey"/>
-            </visual>
-            <collision>
-                <origin xyz="0 0 0" rpy="0 0 0"/>
-                <geometry>
-                    <mesh filename="file://$(find unitree_d1_description)/meshes/Link6.STL"/>
-                </geometry>
-            </collision> -->
+            <inertial>
+                <origin rpy="0 0 0" xyz="0 0 0" />
+                <mass value="0.001" />
+                <inertia
+                    ixx="1e-6" ixy="0" ixz="0"
+                    iyy="1e-6" iyz="0"
+                    izz="1e-6" />
+            </inertial>
         </link>
         <joint name="${prefix}joint_6" type="revolute">
-            <origin xyz="0.0825 -0.0010782 -0.023822" rpy="-1.5708 0 -1.5708"/>
-            <parent link="${prefix}Link5"/>
-            <child link="${prefix}Link6"/>
-            <axis xyz="0 0 -1"/>
+            <origin rpy="-1.5708 0 -1.5708" xyz="0.0825 -0.0010782 -0.023822" />
+            <parent link="${prefix}Link5" />
+            <child link="${prefix}Link6" />
+            <axis xyz="0 0 -1" />
             <limit lower="${min_joint_6_pos}" upper="${max_joint_6_pos}"
                     effort="${joint_6_effort}" velocity="${joint_6_vel}" />
@@ -200,5 +208,5 @@
             <xacro:include filename="$(find unitree_d1_description)/urdf/camera/d435.urdf.xacro" />
             <xacro:d435_camera parent="base_link" prefix="${prefix}">
-                <origin xyz="0.22 -0.60 0" rpy="0 0 0"/>
+                <origin rpy="0 0 0" xyz="0.22 -0.60 0" />
             </xacro:d435_camera>
         </xacro:if>
@@ -209,13 +217,4 @@
         <xacro:include filename="$(find unitree_d1_description)/urdf/ros2_control/unitree_d1_ros2_control.xacro" />
         <xacro:unitree_d1_ros2_control prefix="${prefix}" sim_gazebo="${sim_gazebo}" />
-        <!-- <xacro:if value="${not gripper}">
-            <link name="${prefix}tool_frame"/>
-            <joint name="${prefix}tool_frame_joint" type="fixed">
-                <origin xyz="0 0 0" rpy="0 0 0" />
-                <parent link="${prefix}${last_arm_link}" />
-                <child link="${prefix}tool_frame" />
-                <axis xyz="0 0 0" />
-            </joint>
-        </xacro:if> -->
     </xacro:macro>
 </robot>
