Commit message: reformat URDF for readability

File: gen3_lite/gen3_lite_description/urdf/camera/d435.urdf.xacro (robot description, xacro)
@@ -1,131 +1,137 @@
 <?xml version="1.0"?>
 <robot xmlns:xacro="http://www.ros.org/wiki/xacro">
-  <xacro:macro name="d435_camera" params="*origin parent prefix">
-    <xacro:property name="M_PI" value="3.1415926535897931" />
-    <xacro:property name="d435_cam_width" value="0.090"/>
-    <xacro:property name="d435_cam_height" value="0.025"/>
-    <xacro:property name="d435_cam_depth" value="0.02505"/>
-    <xacro:property name="d435_cam_depth_to_infra1_offset" value="0.0"/>
-    <xacro:property name="d435_cam_depth_to_infra2_offset" value="-0.050"/>
-    <xacro:property name="d435_cam_depth_to_color_offset" value="0.015"/>
-    <xacro:property name="camera_tilt_angle_deg" value="25"/>
-    <link name="${prefix}torso_link">
-      <inertial>
-        <origin xyz="0 0 0.50" />
-        <mass value="2.5" />
-        <inertia ixx="0.8" ixy="0.0" ixz="0.0" iyy="0.8" iyz="0.0" izz="0.8" />
-      </inertial>
-      <visual name="holder">
-        <origin xyz="0 0 0.25" rpy="0 0 0" />
-        <material name="LightGrey">
-          <color rgba="0.7 0.7 0.7 1.0"/>
-        </material>
-        <geometry>
-          <cylinder radius="0.005" length="0.5"/>
-        </geometry>
-      </visual>
-      <visual name="base">
-        <origin xyz="0 0 0" rpy="0 0 0" />
-        <material name="LightGrey">
-          <color rgba="0.7 0.7 0.7 1.0"/>
-        </material>
-        <geometry>
-          <box size="0.15 0.10 0.06" />
-        </geometry>
-      </visual>
-      <collision name="holder">
-        <origin xyz="0 0 0.25" rpy="0 0 0" />
-        <geometry>
-          <cylinder radius="0.005" length="0.6"/>
-        </geometry>
-      </collision>
-      <collision name="base">
-        <origin xyz="0 0 0.0" rpy="0 0 0" />
-        <geometry>
-          <box size="0.15 0.10 0.06" />
-        </geometry>
-      </collision>
-    </link>
-    <joint name="${prefix}base_link_to_torso_link" type="fixed">
-      <parent link="${prefix}${parent}"/>
-      <child link="${prefix}torso_link"/>
-      <xacro:insert_block name="origin" />
-      <!-- <origin xyz="0.22 -0.30 0" rpy="0 0 0"/> -->
-    </joint>
-    <joint name="${prefix}camera_head_joint" type="fixed">
-      <parent link="${prefix}torso_link"/>
-      <child link="${prefix}camera_head_link" />
-      <origin xyz="0 0.01 0.50" rpy="0.0 ${camera_tilt_angle_deg * M_PI / 180} ${M_PI/2}"/>
-    </joint>
-    <link name="${prefix}camera_head_link">
-      <visual>
-        <origin xyz="0 0 0" rpy="${M_PI/2} 0.0 ${M_PI/2}"/>
-        <geometry>
-          <mesh filename="file://$(find gen3_lite_description)/meshes/d435.stl" />
-        </geometry>
-        <material name="aluminum">
-          <color rgba="0.5 0.5 0.5 1"/>
-        </material>
-      </visual>
-      <collision>
-        <origin xyz="0 0 0" rpy="0 0 0"/>
-        <geometry>
-          <box size="${d435_cam_depth} ${d435_cam_width} ${d435_cam_height}"/>
-        </geometry>
-      </collision>
-      <inertial>
-        <mass value="0.072" />
-        <origin xyz="0 0 0" />
-        <inertia ixx="0.003881243" ixy="0.0" ixz="0.0" iyy="0.000498940" iyz="0.0" izz="0.003879257" />
-      </inertial>
-    </link>
-    <joint name="${prefix}camera_head_depth_joint" type="fixed">
-      <origin xyz="0 0 0" rpy="0 0 0"/>
-      <parent link="${prefix}camera_head_link"/>
-      <child link="${prefix}camera_head_depth_frame" />
-    </joint>
-    <link name="${prefix}camera_head_depth_frame"/>
-    <joint name="${prefix}camera_head_depth_optical_joint" type="fixed">
-      <origin xyz="0 0 0" rpy="${-M_PI/2} 0 ${-M_PI/2}" />
-      <parent link="${prefix}camera_head_depth_frame" />
-      <child link="${prefix}camera_head_depth_optical_frame" />
-    </joint>
-    <link name="${prefix}camera_head_depth_optical_frame"/>
-    <joint name="${prefix}camera_head_infra1_joint" type="fixed">
-      <origin xyz="0 ${d435_cam_depth_to_infra1_offset} 0" rpy="0 0 0" />
-      <parent link="${prefix}camera_head_link" />
-      <child link="${prefix}camera_head_infra1_frame" />
-    </joint>
-    <link name="${prefix}camera_head_infra1_frame"/>
-    <joint name="${prefix}camera_head_infra1_optical_joint" type="fixed">
-      <origin xyz="0 0 0" rpy="${-M_PI/2} 0 ${-M_PI/2}" />
-      <parent link="${prefix}camera_head_infra1_frame" />
-      <child link="${prefix}camera_head_infra1_optical_frame" />
-    </joint>
-    <link name="${prefix}camera_head_infra1_optical_frame"/>
-    <joint name="${prefix}camera_head_infra2_joint" type="fixed">
-      <origin xyz="0 ${d435_cam_depth_to_infra2_offset} 0" rpy="0 0 0" />
-      <parent link="${prefix}camera_head_link" />
-      <child link="${prefix}camera_head_infra2_frame" />
-    </joint>
-    <link name="${prefix}camera_head_infra2_frame"/>
-    <joint name="${prefix}camera_head_infra2_optical_joint" type="fixed">
-      <origin xyz="0 0 0" rpy="${-M_PI/2} 0 ${-M_PI/2}" />
-      <parent link="${prefix}camera_head_infra2_frame" />
-      <child link="${prefix}camera_head_infra2_optical_frame" />
-    </joint>
-    <link name="${prefix}camera_head_infra2_optical_frame"/>
-    <joint name="${prefix}camera_head_color_joint" type="fixed">
-      <origin xyz="0 ${d435_cam_depth_to_color_offset} 0" rpy="0 0 0" />
-      <parent link="${prefix}camera_head_link" />
-      <child link="${prefix}camera_head_color_frame" />
-    </joint>
-    <link name="${prefix}camera_head_color_frame"/>
-    <joint name="${prefix}camera_head_color_optical_joint" type="fixed">
-      <origin xyz="0 0 0" rpy="${-M_PI/2} 0 ${-M_PI/2}" />
-      <parent link="${prefix}camera_head_color_frame" />
-      <child link="${prefix}camera_head_color_optical_frame" />
-    </joint>
-    <link name="${prefix}camera_head_color_optical_frame"/>
-  </xacro:macro>
+    <xacro:macro name="d435_camera" params="*origin parent prefix">
+        <xacro:property name="M_PI" value="3.1415926535897931" />
+        <xacro:property name="d435_cam_width" value="0.090"/>
+        <xacro:property name="d435_cam_height" value="0.025"/>
+        <xacro:property name="d435_cam_depth" value="0.02505"/>
+        <xacro:property name="d435_cam_depth_to_infra1_offset" value="0.0"/>
+        <xacro:property name="d435_cam_depth_to_infra2_offset" value="-0.050"/>
+        <xacro:property name="d435_cam_depth_to_color_offset" value="0.015"/>
+        <xacro:property name="camera_tilt_angle_deg" value="25"/>
+        <link name="${prefix}torso_link">
+            <inertial>
+                <origin xyz="0 0 0.50" />
+                <mass value="2.5" />
+                <inertia
+                    ixx="0.8" ixy="0.0" ixz="0.0"
+                    iyy="0.8" iyz="0.0"
+                    izz="0.8" />
+            </inertial>
+            <visual name="holder">
+                <origin rpy="0 0 0" xyz="0 0 0.25" />
+                <material name="LightGrey">
+                    <color rgba="0.7 0.7 0.7 1.0"/>
+                </material>
+                <geometry>
+                    <cylinder radius="0.005" length="0.5"/>
+                </geometry>
+            </visual>
+            <visual name="base">
+                <origin rpy="0 0 0" xyz="0 0 0" />
+                <material name="LightGrey">
+                    <color rgba="0.7 0.7 0.7 1.0"/>
+                </material>
+                <geometry>
+                    <box size="0.15 0.10 0.06" />
+                </geometry>
+            </visual>
+            <collision name="holder">
+                <origin rpy="0 0 0" xyz="0 0 0.25" />
+                <geometry>
+                <cylinder radius="0.005" length="0.6"/>
+                </geometry>
+            </collision>
+            <collision name="base">
+                <origin rpy="0 0 0" xyz="0 0 0.0" />
+                <geometry>
+                <box size="0.15 0.10 0.06" />
+                </geometry>
+            </collision>
+        </link>
+        <joint name="${prefix}base_link_to_torso_link" type="fixed">
+            <parent link="${prefix}${parent}"/>
+            <child link="${prefix}torso_link"/>
+            <xacro:insert_block name="origin" />
+            <!-- <origin rpy="0 0 0" xyz="0.22 -0.30 0" /> -->
+        </joint>
+        <joint name="${prefix}camera_head_joint" type="fixed">
+            <parent link="${prefix}torso_link"/>
+            <child link="${prefix}camera_head_link" />
+            <origin rpy="0.0 ${camera_tilt_angle_deg * M_PI / 180} ${M_PI/2}" xyz="0 0.01 0.50" />
+        </joint>
+        <link name="${prefix}camera_head_link">
+            <inertial>
+                <origin xyz="0 0 0" />
+                <mass value="0.072" />
+                <inertia
+                    ixx="0.003881243" ixy="0.0" ixz="0.0"
+                    iyy="0.000498940" iyz="0.0"
+                    izz="0.003879257" />
+            </inertial>
+            <visual>
+                <origin rpy="${M_PI/2} 0.0 ${M_PI/2}" xyz="0 0 0" />
+                <geometry>
+                    <mesh filename="file://$(find gen3_lite_description)/meshes/d435.stl" />
+                </geometry>
+                <material name="aluminum">
+                    <color rgba="0.5 0.5 0.5 1"/>
+                </material>
+            </visual>
+            <collision>
+                <origin rpy="0 0 0" xyz="0 0 0" />
+                <geometry>
+                    <box size="${d435_cam_depth} ${d435_cam_width} ${d435_cam_height}"/>
+                </geometry>
+            </collision>
+        </link>
+        <joint name="${prefix}camera_head_depth_joint" type="fixed">
+            <origin rpy="0 0 0" xyz="0 0 0" />
+            <parent link="${prefix}camera_head_link"/>
+            <child link="${prefix}camera_head_depth_frame" />
+        </joint>
+        <link name="${prefix}camera_head_depth_frame"/>
+        <joint name="${prefix}camera_head_depth_optical_joint" type="fixed">
+            <origin rpy="${-M_PI/2} 0 ${-M_PI/2}" xyz="0 0 0" />
+            <parent link="${prefix}camera_head_depth_frame" />
+            <child link="${prefix}camera_head_depth_optical_frame" />
+        </joint>
+        <link name="${prefix}camera_head_depth_optical_frame"/>
+        <joint name="${prefix}camera_head_infra1_joint" type="fixed">
+            <origin rpy="0 0 0" xyz="0 ${d435_cam_depth_to_infra1_offset} 0" />
+            <parent link="${prefix}camera_head_link" />
+            <child link="${prefix}camera_head_infra1_frame" />
+        </joint>
+        <link name="${prefix}camera_head_infra1_frame"/>
+        <joint name="${prefix}camera_head_infra1_optical_joint" type="fixed">
+            <origin rpy="${-M_PI/2} 0 ${-M_PI/2}" xyz="0 0 0" />
+            <parent link="${prefix}camera_head_infra1_frame" />
+            <child link="${prefix}camera_head_infra1_optical_frame" />
+        </joint>
+        <link name="${prefix}camera_head_infra1_optical_frame"/>
+        <joint name="${prefix}camera_head_infra2_joint" type="fixed">
+            <origin rpy="0 0 0" xyz="0 ${d435_cam_depth_to_infra2_offset} 0" />
+            <parent link="${prefix}camera_head_link" />
+            <child link="${prefix}camera_head_infra2_frame" />
+        </joint>
+        <link name="${prefix}camera_head_infra2_frame"/>
+        <joint name="${prefix}camera_head_infra2_optical_joint" type="fixed">
+            <origin rpy="${-M_PI/2} 0 ${-M_PI/2}" xyz="0 0 0" />
+            <parent link="${prefix}camera_head_infra2_frame" />
+            <child link="${prefix}camera_head_infra2_optical_frame" />
+        </joint>
+        <link name="${prefix}camera_head_infra2_optical_frame"/>
+        <joint name="${prefix}camera_head_color_joint" type="fixed">
+            <origin rpy="0 0 0" xyz="0 ${d435_cam_depth_to_color_offset} 0" />
+            <parent link="${prefix}camera_head_link" />
+            <child link="${prefix}camera_head_color_frame" />
+        </joint>
+        <link name="${prefix}camera_head_color_frame"/>
+        <joint name="${prefix}camera_head_color_optical_joint" type="fixed">
+            <origin rpy="${-M_PI/2} 0 ${-M_PI/2}" xyz="0 0 0" />
+            <parent link="${prefix}camera_head_color_frame" />
+            <child link="${prefix}camera_head_color_optical_frame" />
+        </joint>
+        <link name="${prefix}camera_head_color_optical_frame"/>
+    </xacro:macro>
 </robot>

File: gen3_lite/gen3_lite_description/urdf/gen3_lite.urdf.xacro (robot description, xacro)
@@ -2,10 +2,7 @@
 <robot name="$(arg name)" xmlns:xacro="http://ros.org/wiki/xacro">
     <!-- Arguments -->
-    <xacro:arg name="moveit_active" default="false" />
-    <xacro:arg name="sim_gazebo" default="true" />
-    <xacro:arg name="use_camera" default="true" />
-    <xacro:arg name="parent" default="world"/>
+    <xacro:arg name="sim_gazebo" default="false" />
+    <xacro:arg name="use_camera" default="false" />
     <xacro:arg name="prefix" default=""/>
-    <xacro:arg name="arm" default="gen3_lite" />
     <xacro:arg name="gripper" default="" />
     <xacro:arg name="joint_limits" default="$(find gen3_lite_description)/config/joint_limits.yaml" />
@@ -28,17 +25,20 @@
     <xacro:include filename="$(find gen3_lite_description)/urdf/macros.urdf.xacro" />
     <link name="world"/>
-    <xacro:load_arm parent="$(arg parent)"
+    <xacro:load_arm
+        parent="world"
+        prefix="$(arg prefix)"
+        sim_gazebo="$(arg sim_gazebo)"
+        gripper="$(arg gripper)"
+        use_camera="$(arg use_camera)">
+        <origin rpy="0 0 0" xyz="0 0 0" />
+    </xacro:load_arm>
+    <xacro:property name="gripper_pkg" value="$(arg gripper)_description" />
+    <xacro:unless value="${not '$(arg gripper)'}">
+        <xacro:include filename="$(find ${gripper_pkg})/urdf/$(arg gripper)_macro.urdf.xacro" />
+        <xacro:load_gripper
+            parent="${last_arm_link}"
             prefix="$(arg prefix)"
-            sim_gazebo="$(arg sim_gazebo)"
-            gripper="$(arg gripper)"
-            use_camera="$(arg use_camera)" >
-        <origin xyz="0 0 0" rpy="0 0 0" />
-    </xacro:load_arm>
-    <xacro:include filename="$(find kinova_2f_lite_description)/urdf/kinova_2f_lite_macro.urdf.xacro" />
-    <xacro:unless value="${not '$(arg gripper)'}" >
-        <xacro:load_gripper parent="${last_arm_link}"
-                prefix="$(arg prefix)"
-                sim_gazebo="$(arg sim_gazebo)" >
-            <origin xyz="0 0 0" rpy="0 0 0" />
+            sim_gazebo="$(arg sim_gazebo)">
+            <origin rpy="0 0 0" xyz="0 0 0" />
         </xacro:load_gripper>
     </xacro:unless>
