Commit message: reformat URDF for readability

File: gen3_lite/gen3_lite_description/urdf/gen3_lite_macro.urdf.xacro (robot description, xacro)
@@ -3,5 +3,11 @@
     <!-- Propagate last link name information because it is the gripper's parent link -->
     <xacro:property name="last_arm_link" value="dummy_link"/>
-    <xacro:macro name="load_arm" params="*origin parent prefix sim_gazebo gripper use_camera">
+    <xacro:macro name="load_arm" params="
+        *origin
+        parent
+        prefix
+        sim_gazebo
+        gripper
+        use_camera">
         <joint name="${prefix}base_joint" type="fixed">
             <xacro:insert_block name="origin" />
@@ -11,33 +17,39 @@
         <link name="${prefix}base_link">
             <inertial>
-                <origin xyz="0.00244324 0.00015573 0.08616742" rpy="0 0 0" />
+                <origin rpy="0 0 0" xyz="0.00244324 0.00015573 0.08616742" />
                 <mass value="1.14608471" />
-                <inertia ixx="0.00335854" ixy="3.9E-07" ixz="0.00010989" iyy="0.003311" iyz="1.91E-06" izz="0.00077158" />
+                <inertia
+                    ixx="0.00335854" ixy="3.9E-07" ixz="0.00010989"
+                    iyy="0.003311" iyz="1.91E-06"
+                    izz="0.00077158" />
+            </inertial>
+            <visual>
+                <origin rpy="0 0 0" xyz="0 0 0" />
+                <geometry>
+                    <mesh filename="file://$(find gen3_lite_description)/meshes/base_link.STL" />
+                </geometry>
+                <material name="">
+                    <color rgba="0.803 0.824 0.820 1" />
+                </material>
+            </visual>
+            <collision>
+                <origin rpy="0 0 0" xyz="0 0 0" />
+                <geometry>
+                    <mesh filename="file://$(find gen3_lite_description)/meshes/base_link.STL" />
+                </geometry>
+            </collision>
+        </link>
+        <link name="${prefix}shoulder_link">
+            <inertial>
+                <origin rpy="0 0 0" xyz="2.477E-05 0.02213531 0.09937686" />
+                <mass value="0.95974404" />
+                <inertia
+                    ixx="0.00165947" ixy="2E-08" ixz="3.6E-07"
+                    iyy="0.00140355" iyz="0.00034927"
+                    izz="0.00089493" />
             </inertial>
             <visual>
                 <origin xyz="0 0 0" rpy="0 0 0" />
                 <geometry>
-                    <mesh filename="file://$(find gen3_lite_description)/meshes/base_link.STL" />
-                </geometry>
-                <material name="">
-                    <color rgba="0.803 0.824 0.820 1" />
-                </material>
-            </visual>
-            <collision>
-                <origin xyz="0 0 0" rpy="0 0 0" />
-                <geometry>
-                    <mesh filename="file://$(find gen3_lite_description)/meshes/base_link.STL" />
-                </geometry>
-            </collision>
-        </link>
-        <link name="${prefix}shoulder_link">
-            <inertial>
-                <origin xyz="2.477E-05 0.02213531 0.09937686" rpy="0 0 0" />
-                <mass value="0.95974404" />
-                <inertia ixx="0.00165947" ixy="2E-08" ixz="3.6E-07" iyy="0.00140355" iyz="0.00034927" izz="0.00089493" />
-            </inertial>
-            <visual>
-                <origin xyz="0 0 0" rpy="0 0 0" />
-                <geometry>
                     <mesh filename="file://$(find gen3_lite_description)/meshes/shoulder_link.STL" />
                 </geometry>
@@ -47,5 +59,5 @@
             </visual>
             <collision>
-                <origin xyz="0 0 0" rpy="0 0 0" />
+                <origin rpy="0 0 0" xyz="0 0 0" />
                 <geometry>
                     <mesh filename="file://$(find gen3_lite_description)/meshes/shoulder_link.STL" />
@@ -54,5 +66,5 @@
         </link>
         <joint name="${prefix}joint_1" type="revolute">
-            <origin xyz="0 0 0.12825" rpy="0 0 0" />
+            <origin rpy="0 0 0" xyz="0 0 0.12825" />
             <parent link="${prefix}base_link" />
             <child link="${prefix}shoulder_link" />
@@ -64,10 +76,13 @@
         <link name="${prefix}arm_link">
             <inertial>
-                <origin xyz="0.02998299 0.21154808 0.0453031" rpy="0 0 0" />
+                <origin rpy="0 0 0" xyz="0.02998299 0.21154808 0.0453031" />
                 <mass value="1.17756164" />
-                <inertia ixx="0.01149277" ixy="1E-06" ixz="1.6E-07" iyy="0.00102851" iyz="0.00140765" izz="0.01133492" />
-            </inertial>
-            <visual>
-                <origin xyz="0 0 0" rpy="0 0 0" />
+                <inertia
+                    ixx="0.01149277" ixy="1E-06" ixz="1.6E-07"
+                    iyy="0.00102851" iyz="0.00140765"
+                    izz="0.01133492" />
+            </inertial>
+            <visual>
+                <origin rpy="0 0 0" xyz="0 0 0" />
                 <geometry>
                     <mesh filename="file://$(find gen3_lite_description)/meshes/arm_link.STL" />
@@ -78,5 +93,5 @@
             </visual>
             <collision>
-                <origin xyz="0 0 0" rpy="0 0 0" />
+                <origin rpy="0 0 0" xyz="0 0 0" />
                 <geometry>
                     <mesh filename="file://$(find gen3_lite_description)/meshes/arm_link.STL" />
@@ -85,5 +100,5 @@
         </link>
         <joint name="${prefix}joint_2" type="revolute">
-            <origin xyz="0 -0.03 0.115" rpy="1.5708 0 0" />
+            <origin rpy="1.5708 0 0" xyz="0 -0.03 0.115" />
             <parent link="${prefix}shoulder_link" />
             <child link="${prefix}arm_link" />
@@ -95,10 +110,13 @@
         <link name="${prefix}forearm_link">
             <inertial>
-                <origin xyz="0.0301559 0.09502206 0.0073555" rpy="0 0 0" />
+                <origin rpy="0 0 0" xyz="0.0301559 0.09502206 0.0073555" />
                 <mass value="0.59767669" />
-                <inertia ixx="0.00163256" ixy="7.11E-06" ixz="1.54E-06" iyy="0.00029798" iyz="9.587E-05" izz="0.00169091" />
-            </inertial>
-            <visual>
-                <origin xyz="0 0 0" rpy="0 0 0" />
+                <inertia
+                    ixx="0.00163256" ixy="7.11E-06" ixz="1.54E-06"
+                    iyy="0.00029798" iyz="9.587E-05"
+                    izz="0.00169091" />
+            </inertial>
+            <visual>
+                <origin rpy="0 0 0" xyz="0 0 0" />
                 <geometry>
                     <mesh filename="file://$(find gen3_lite_description)/meshes/forearm_link.STL" />
@@ -109,5 +127,5 @@
             </visual>
             <collision>
-                <origin xyz="0 0 0" rpy="0 0 0" />
+                <origin rpy="0 0 0" xyz="0 0 0" />
                 <geometry>
                     <mesh filename="file://$(find gen3_lite_description)/meshes/forearm_link.STL" />
@@ -116,5 +134,5 @@
         </link>
         <joint name="${prefix}joint_3" type="revolute">
-            <origin xyz="0 0.28 0" rpy="-3.1416 0 0" />
+            <origin rpy="-3.1416 0 0" xyz="0 0.28 0" />
             <parent link="${prefix}arm_link" />
             <child link="${prefix}forearm_link" />
@@ -126,10 +144,13 @@
         <link name="${prefix}lower_wrist_link">
             <inertial>
-                <origin xyz="0.00575149 0.01000443 0.08719207" rpy="0 0 0" />
+                <origin rpy="0 0 0" xyz="0.00575149 0.01000443 0.08719207" />
                 <mass value="0.52693412" />
-                <inertia ixx="0.00069098" ixy="2.4E-07" ixz="0.00016483" iyy="0.00078519" iyz="7.4E-07" izz="0.00034115" />
-            </inertial>
-            <visual>
-                <origin xyz="0 0 0" rpy="0 0 0" />
+                <inertia
+                    ixx="0.00069098" ixy="2.4E-07" ixz="0.00016483"
+                    iyy="0.00078519" iyz="7.4E-07"
+                    izz="0.00034115" />
+            </inertial>
+            <visual>
+                <origin rpy="0 0 0" xyz="0 0 0" />
                 <geometry>
                     <mesh filename="file://$(find gen3_lite_description)/meshes/lower_wrist_link.STL" />
@@ -140,5 +161,5 @@
             </visual>
             <collision>
-                <origin xyz="0 0 0" rpy="0 0 0" />
+                <origin rpy="0 0 0" xyz="0 0 0" />
                 <geometry>
                     <mesh filename="file://$(find gen3_lite_description)/meshes/lower_wrist_link.STL" />
@@ -147,5 +168,5 @@
         </link>
         <joint name="${prefix}joint_4" type="revolute">
-            <origin xyz="0 -0.14 0.02" rpy="1.5708 0 0" />
+            <origin rpy="1.5708 0 0" xyz="0 -0.14 0.02" />
             <parent link="${prefix}forearm_link" />
             <child link="${prefix}lower_wrist_link" />
@@ -157,10 +178,13 @@
         <link name="${prefix}upper_wrist_link">
             <inertial>
-                <origin xyz="0.08056517 0.00980409 0.01872799" rpy="0 0 0" />
+                <origin rpy="0 0 0" xyz="0.08056517 0.00980409 0.01872799" />
                 <mass value="0.58097325" />
-                <inertia ixx="0.00021268" ixy="5.21E-06" ixz="2.91E-06" iyy="0.00106371" iyz="1.1E-07" izz="0.00108465" />
-            </inertial>
-            <visual>
-                <origin xyz="0 0 0" rpy="0 0 0" />
+                <inertia
+                    ixx="0.00021268" ixy="5.21E-06" ixz="2.91E-06"
+                    iyy="0.00106371" iyz="1.1E-07"
+                    izz="0.00108465" />
+            </inertial>
+            <visual>
+                <origin rpy="0 0 0" xyz="0 0 0" />
                 <geometry>
                     <mesh filename="file://$(find gen3_lite_description)/meshes/upper_wrist_link.STL" />
@@ -171,5 +195,5 @@
             </visual>
             <collision>
-                <origin xyz="0 0 0" rpy="0 0 0" />
+                <origin rpy="0 0 0" xyz="0 0 0" />
                 <geometry>
                     <mesh filename="file://$(find gen3_lite_description)/meshes/upper_wrist_link.STL" />
@@ -178,5 +202,5 @@
         </link>
         <joint name="${prefix}joint_5" type="revolute">
-            <origin xyz="0.0285 0 0.105" rpy="0 1.5708 0" />
+            <origin rpy="0 1.5708 0" xyz="0.0285 0 0.105" />
             <parent link="${prefix}lower_wrist_link" />
             <child link="${prefix}upper_wrist_link" />
@@ -188,11 +212,14 @@
         <link name="${prefix}end_effector_link">
             <inertial>
-                <origin xyz="0 0 0" rpy="0 0 0" />
-                <mass value="0.01" />
-                <inertia ixx="1e-6" ixy="0" ixz="0" iyy="1e-6" iyz="0" izz="1e-6" />
+                <origin rpy="0 0 0" xyz="0 0 0" />
+                <mass value="0.001" />
+                <inertia
+                    ixx="1e-6" ixy="0" ixz="0"
+                    iyy="1e-6" iyz="0"
+                    izz="1e-6" />
             </inertial>
         </link>
         <joint name="${prefix}joint_6" type="revolute">
-            <origin xyz="-0.105 0 0.0285" rpy="0 -1.5708 0" />
+            <origin rpy="0 -1.5708 0" xyz="-0.105 0 0.0285" />
             <parent link="${prefix}upper_wrist_link" />
             <child link="${prefix}end_effector_link" />
@@ -204,5 +231,5 @@
         <link name="${prefix}dummy_link" />
         <joint name="${prefix}end_effector" type="fixed">
-            <origin xyz="0 0 0" rpy="0 0 0" />
+            <origin rpy="0 0 0" xyz="0 0 0" />
             <parent link="${prefix}end_effector_link" />
             <child link="${prefix}dummy_link" />
@@ -213,5 +240,5 @@
             <xacro:include filename="$(find gen3_lite_description)/urdf/camera/d435.urdf.xacro" />
             <xacro:d435_camera parent="base_link" prefix="${prefix}">
-                <origin xyz="0.22 -0.30 0" rpy="0 0 0"/>
+                <origin rpy="0 0 0" xyz="0.22 -0.30 0" />
             </xacro:d435_camera>
         </xacro:if>
@@ -225,5 +252,5 @@
             <link name="${prefix}tool_frame"/>
             <joint name="${prefix}tool_frame_joint" type="fixed">
-                <origin xyz="0 0 0" rpy="0 0 0" />
+                <origin rpy="0 0 0" xyz="0 0 0" />
                 <parent link="${prefix}${last_arm_link}" />
                 <child link="${prefix}tool_frame" />

File: gen3_lite/gen3_lite_description/urdf/gz/gen3_lite.gazebo.xacro (robot description, xacro)
@@ -1,54 +1,54 @@
 <?xml version="1.0"?>
 <robot xmlns:xacro="http://ros.org/wiki/xacro">
-  <xacro:macro name="gen3_lite_gazebo" params="parent prefix use_camera">
-    <gazebo reference="${prefix}base_link">
-        <material>Kortex/Gray</material>
-    </gazebo>
-    <gazebo reference="${prefix}shoulder_link">
-        <material>Kortex/Gray</material>
-    </gazebo>
-    <gazebo reference="${prefix}arm_link">
-        <material>Kortex/Gray</material>
-    </gazebo>
-    <gazebo reference="${prefix}forearm_link">
-        <material>Kortex/Gray</material>
-    </gazebo>
-    <gazebo reference="${prefix}lower_wrist_link">
-        <material>Kortex/Gray</material>
-    </gazebo>
-    <gazebo reference="${prefix}upper_wrist_link">
-        <material>Kortex/Gray</material>
-    </gazebo>
-    <xacro:if value="${use_camera}">
-      <gazebo reference="${prefix}camera_head_link">
-        <sensor name="${prefix}camera_head" type="rgbd_camera">
-          <camera>
-            <horizontal_fov>1.5184</horizontal_fov>
-            <image>
-              <width>424</width>
-              <height>240</height>
-            </image>
-            <clip>
-              <near>0.05</near>
-              <far>1.5</far>
-            </clip>
-          </camera>
-          <always_on>1</always_on>
-          <gz_frame_id>${prefix}camera_head_link</gz_frame_id>
-          <topic>${prefix}camera_head</topic>
-          <update_rate>5</update_rate>
-          <visualize>true</visualize>
-        </sensor>
-      </gazebo>
-    </xacro:if>
-    <!-- ROS2 CONTROL -->
-    <!-- condition to avoid conflicts when launching the arm as an accessory. -->
-    <xacro:if value="${parent == 'world'}">
-      <gazebo>
-        <plugin filename="gz_ros2_control-system" name="gz_ros2_control::GazeboSimROS2ControlPlugin">
-          <parameters>$(find arms_bringup)/config/ros2_control.yaml</parameters>
-        </plugin>
-      </gazebo>
-    </xacro:if>
-  </xacro:macro>
+    <xacro:macro name="gen3_lite_gazebo" params="parent prefix use_camera">
+        <gazebo reference="${prefix}base_link">
+            <material>Kortex/Gray</material>
+        </gazebo>
+        <gazebo reference="${prefix}shoulder_link">
+            <material>Kortex/Gray</material>
+        </gazebo>
+        <gazebo reference="${prefix}arm_link">
+            <material>Kortex/Gray</material>
+        </gazebo>
+        <gazebo reference="${prefix}forearm_link">
+            <material>Kortex/Gray</material>
+        </gazebo>
+        <gazebo reference="${prefix}lower_wrist_link">
+            <material>Kortex/Gray</material>
+        </gazebo>
+        <gazebo reference="${prefix}upper_wrist_link">
+            <material>Kortex/Gray</material>
+        </gazebo>
+        <xacro:if value="${use_camera}">
+        <gazebo reference="${prefix}camera_head_link">
+            <sensor name="${prefix}camera_head" type="rgbd_camera">
+                <camera>
+                    <horizontal_fov>1.5184</horizontal_fov>
+                    <image>
+                        <width>424</width>
+                        <height>240</height>
+                    </image>
+                    <clip>
+                        <near>0.05</near>
+                        <far>1.5</far>
+                    </clip>
+                </camera>
+                <always_on>1</always_on>
+                <gz_frame_id>${prefix}camera_head_link</gz_frame_id>
+                <topic>${prefix}camera_head</topic>
+                <update_rate>5</update_rate>
+                <visualize>true</visualize>
+            </sensor>
+        </gazebo>
+        </xacro:if>
+        <!-- ROS2 CONTROL -->
+        <!-- condition to avoid conflicts when launching the arm as an accessory. -->
+        <xacro:if value="${parent == 'world'}">
+            <gazebo>
+                <plugin filename="gz_ros2_control-system" name="gz_ros2_control::GazeboSimROS2ControlPlugin">
+                    <parameters>$(find arms_bringup)/config/ros2_control.yaml</parameters>
+                </plugin>
+            </gazebo>
+        </xacro:if>
+    </xacro:macro>
 </robot>
