Commit message: reformat URDF for readability

File: gen3_lite/gen3_lite_description/urdf/ros2_control/gen3_lite_ros2_control.xacro (robot description, xacro)
@@ -1,78 +1,78 @@
 <?xml version="1.0"?>
 <robot xmlns:xacro="http://ros.org/wiki/xacro">
-  <xacro:macro name="gen3_lite_ros2_control" params="prefix sim_gazebo" >
-    <ros2_control name="ArmHardwareInterface" type="system">
-        <xacro:if value="${sim_gazebo}">
-            <hardware>
-                <plugin>gz_ros2_control/GazeboSimSystem</plugin>
-            </hardware>
-        </xacro:if>
-        <joint name="${prefix}joint_1">
-            <command_interface name="position">
-                <param name="min">${min_joint_1_pos}</param>
-                <param name="max">${max_joint_1_pos}</param>
-            </command_interface>
-            <state_interface name="position">
-                <param name="initial_value">${joint_1_initial}</param>
-            </state_interface>
-            <state_interface name="velocity"/>
-            <state_interface name="effort"/>
-        </joint>
-        <joint name="${prefix}joint_2">
-            <command_interface name="position">
-                <param name="min">${min_joint_2_pos}</param>
-                <param name="max">${max_joint_2_pos}</param>
-            </command_interface>
-            <state_interface name="position">
-                <param name="initial_value">${joint_2_initial}</param>
-            </state_interface>
-            <state_interface name="velocity"/>
-            <state_interface name="effort"/>
-        </joint>
-        <joint name="${prefix}joint_3">
-            <command_interface name="position">
-                <param name="min">${min_joint_3_pos}</param>
-                <param name="max">${max_joint_3_pos}</param>
-            </command_interface>
-            <state_interface name="position">
-                <param name="initial_value">${joint_3_initial}</param>
-            </state_interface>
-            <state_interface name="velocity"/>
-            <state_interface name="effort"/>
-        </joint>
-        <joint name="${prefix}joint_4">
-            <command_interface name="position">
-                <param name="min">${min_joint_4_pos}</param>
-                <param name="max">${max_joint_4_pos}</param>
-            </command_interface>
-            <state_interface name="position">
-                <param name="initial_value">${joint_4_initial}</param>
-            </state_interface>
-            <state_interface name="velocity"/>
-            <state_interface name="effort"/>
-        </joint>
-        <joint name="${prefix}joint_5">
-            <command_interface name="position">
-                <param name="min">${min_joint_5_pos}</param>
-                <param name="max">${max_joint_5_pos}</param>
-            </command_interface>
-            <state_interface name="position">
-                <param name="initial_value">${joint_5_initial}</param>
-            </state_interface>
-            <state_interface name="velocity"/>
-            <state_interface name="effort"/>
-        </joint>
-        <joint name="${prefix}joint_6">
-            <command_interface name="position">
-                <param name="min">${min_joint_6_pos}</param>
-                <param name="max">${max_joint_6_pos}</param>
-            </command_interface>
-            <state_interface name="position">
-                <param name="initial_value">${joint_6_initial}</param>
-            </state_interface>
-            <state_interface name="velocity"/>
-            <state_interface name="effort"/>
-        </joint>
-    </ros2_control>
-  </xacro:macro>
+    <xacro:macro name="gen3_lite_ros2_control" params="prefix sim_gazebo" >
+        <ros2_control name="ArmHardwareInterface" type="system">
+            <xacro:if value="${sim_gazebo}">
+                <hardware>
+                    <plugin>gz_ros2_control/GazeboSimSystem</plugin>
+                </hardware>
+            </xacro:if>
+            <joint name="${prefix}joint_1">
+                <command_interface name="position">
+                    <param name="min">${min_joint_1_pos}</param>
+                    <param name="max">${max_joint_1_pos}</param>
+                </command_interface>
+                <state_interface name="position">
+                    <param name="initial_value">${joint_1_initial}</param>
+                </state_interface>
+                <state_interface name="velocity"/>
+                <state_interface name="effort"/>
+            </joint>
+            <joint name="${prefix}joint_2">
+                <command_interface name="position">
+                    <param name="min">${min_joint_2_pos}</param>
+                    <param name="max">${max_joint_2_pos}</param>
+                </command_interface>
+                <state_interface name="position">
+                    <param name="initial_value">${joint_2_initial}</param>
+                </state_interface>
+                <state_interface name="velocity"/>
+                <state_interface name="effort"/>
+            </joint>
+            <joint name="${prefix}joint_3">
+                <command_interface name="position">
+                    <param name="min">${min_joint_3_pos}</param>
+                    <param name="max">${max_joint_3_pos}</param>
+                </command_interface>
+                <state_interface name="position">
+                    <param name="initial_value">${joint_3_initial}</param>
+                </state_interface>
+                <state_interface name="velocity"/>
+                <state_interface name="effort"/>
+            </joint>
+            <joint name="${prefix}joint_4">
+                <command_interface name="position">
+                    <param name="min">${min_joint_4_pos}</param>
+                    <param name="max">${max_joint_4_pos}</param>
+                </command_interface>
+                <state_interface name="position">
+                    <param name="initial_value">${joint_4_initial}</param>
+                </state_interface>
+                <state_interface name="velocity"/>
+                <state_interface name="effort"/>
+            </joint>
+            <joint name="${prefix}joint_5">
+                <command_interface name="position">
+                    <param name="min">${min_joint_5_pos}</param>
+                    <param name="max">${max_joint_5_pos}</param>
+                </command_interface>
+                <state_interface name="position">
+                    <param name="initial_value">${joint_5_initial}</param>
+                </state_interface>
+                <state_interface name="velocity"/>
+                <state_interface name="effort"/>
+            </joint>
+            <joint name="${prefix}joint_6">
+                <command_interface name="position">
+                    <param name="min">${min_joint_6_pos}</param>
+                    <param name="max">${max_joint_6_pos}</param>
+                </command_interface>
+                <state_interface name="position">
+                    <param name="initial_value">${joint_6_initial}</param>
+                </state_interface>
+                <state_interface name="velocity"/>
+                <state_interface name="effort"/>
+            </joint>
+        </ros2_control>
+    </xacro:macro>
 </robot>

Commit message: update meshes

File: gen3_lite/gen3_lite_description/urdf/camera/d435.urdf.xacro (robot description, xacro)
@@ -73,5 +73,5 @@
                 <origin rpy="${M_PI/2} 0.0 ${M_PI/2}" xyz="0 0 0" />
                 <geometry>
-                    <mesh filename="file://$(find gen3_lite_description)/meshes/d435.stl" />
+                    <mesh filename="package://gen3_lite_description/meshes/d435.stl" />
                 </geometry>
                 <material name="aluminum">

File: gen3_lite/gen3_lite_description/urdf/gen3_lite.urdf.xacro (robot description, xacro)
@@ -23,5 +23,4 @@
     <xacro:arg name="use_external_cable" default="false" />
     <xacro:include filename="$(find gen3_lite_description)/urdf/gen3_lite_macro.urdf.xacro" />
-    <xacro:include filename="$(find gen3_lite_description)/urdf/macros.urdf.xacro" />
     <link name="world"/>
     <xacro:load_arm

File: gen3_lite/gen3_lite_description/urdf/gen3_lite_macro.urdf.xacro (robot description, xacro)
@@ -3,4 +3,5 @@
     <!-- Propagate last link name information because it is the gripper's parent link -->
     <xacro:property name="last_arm_link" value="dummy_link"/>
+    <xacro:include filename="$(find gen3_lite_description)/urdf/macros.urdf.xacro" />
     <xacro:macro name="load_arm" params="
         *origin
@@ -27,14 +28,14 @@
                 <origin rpy="0 0 0" xyz="0 0 0" />
                 <geometry>
-                    <mesh filename="file://$(find gen3_lite_description)/meshes/base_link.STL" />
-                </geometry>
-                <material name="">
-                    <color rgba="0.803 0.824 0.820 1" />
-                </material>
-            </visual>
-            <collision>
-                <origin rpy="0 0 0" xyz="0 0 0" />
-                <geometry>
-                    <mesh filename="file://$(find gen3_lite_description)/meshes/base_link.STL" />
+                    <mesh filename="package://gen3_lite_description/meshes/base_link.STL" />
+                </geometry>
+                <material name="">
+                    <color rgba="0.803 0.824 0.820 1" />
+                </material>
+            </visual>
+            <collision>
+                <origin rpy="0 0 0" xyz="0 0 0" />
+                <geometry>
+                    <mesh filename="package://gen3_lite_description/meshes/base_link.STL" />
                 </geometry>
             </collision>
@@ -52,14 +53,14 @@
                 <origin xyz="0 0 0" rpy="0 0 0" />
                 <geometry>
-                    <mesh filename="file://$(find gen3_lite_description)/meshes/shoulder_link.STL" />
-                </geometry>
-                <material name="">
-                    <color rgba="0.803 0.824 0.820 1" />
-                </material>
-            </visual>
-            <collision>
-                <origin rpy="0 0 0" xyz="0 0 0" />
-                <geometry>
-                    <mesh filename="file://$(find gen3_lite_description)/meshes/shoulder_link.STL" />
+                    <mesh filename="package://gen3_lite_description/meshes/shoulder_link.STL" />
+                </geometry>
+                <material name="">
+                    <color rgba="0.803 0.824 0.820 1" />
+                </material>
+            </visual>
+            <collision>
+                <origin rpy="0 0 0" xyz="0 0 0" />
+                <geometry>
+                    <mesh filename="package://gen3_lite_description/meshes/shoulder_link.STL" />
                 </geometry>
             </collision>
@@ -86,14 +87,14 @@
                 <origin rpy="0 0 0" xyz="0 0 0" />
                 <geometry>
-                    <mesh filename="file://$(find gen3_lite_description)/meshes/arm_link.STL" />
-                </geometry>
-                <material name="">
-                    <color rgba="0.803 0.824 0.820 1" />
-                </material>
-            </visual>
-            <collision>
-                <origin rpy="0 0 0" xyz="0 0 0" />
-                <geometry>
-                    <mesh filename="file://$(find gen3_lite_description)/meshes/arm_link.STL" />
+                    <mesh filename="package://gen3_lite_description/meshes/arm_link.STL" />
+                </geometry>
+                <material name="">
+                    <color rgba="0.803 0.824 0.820 1" />
+                </material>
+            </visual>
+            <collision>
+                <origin rpy="0 0 0" xyz="0 0 0" />
+                <geometry>
+                    <mesh filename="package://gen3_lite_description/meshes/arm_link.STL" />
                 </geometry>
             </collision>
@@ -120,14 +121,14 @@
                 <origin rpy="0 0 0" xyz="0 0 0" />
                 <geometry>
-                    <mesh filename="file://$(find gen3_lite_description)/meshes/forearm_link.STL" />
-                </geometry>
-                <material name="">
-                    <color rgba="0.803 0.824 0.820 1" />
-                </material>
-            </visual>
-            <collision>
-                <origin rpy="0 0 0" xyz="0 0 0" />
-                <geometry>
-                    <mesh filename="file://$(find gen3_lite_description)/meshes/forearm_link.STL" />
+                    <mesh filename="package://gen3_lite_description/meshes/forearm_link.STL" />
+                </geometry>
+                <material name="">
+                    <color rgba="0.803 0.824 0.820 1" />
+                </material>
+            </visual>
+            <collision>
+                <origin rpy="0 0 0" xyz="0 0 0" />
+                <geometry>
+                    <mesh filename="package://gen3_lite_description/meshes/forearm_link.STL" />
                 </geometry>
             </collision>
@@ -154,14 +155,14 @@
                 <origin rpy="0 0 0" xyz="0 0 0" />
                 <geometry>
-                    <mesh filename="file://$(find gen3_lite_description)/meshes/lower_wrist_link.STL" />
-                </geometry>
-                <material name="">
-                    <color rgba="0.803 0.824 0.820 1" />
-                </material>
-            </visual>
-            <collision>
-                <origin rpy="0 0 0" xyz="0 0 0" />
-                <geometry>
-                    <mesh filename="file://$(find gen3_lite_description)/meshes/lower_wrist_link.STL" />
+                    <mesh filename="package://gen3_lite_description/meshes/lower_wrist_link.STL" />
+                </geometry>
+                <material name="">
+                    <color rgba="0.803 0.824 0.820 1" />
+                </material>
+            </visual>
+            <collision>
+                <origin rpy="0 0 0" xyz="0 0 0" />
+                <geometry>
+                    <mesh filename="package://gen3_lite_description/meshes/lower_wrist_link.STL" />
                 </geometry>
             </collision>
@@ -188,14 +189,14 @@
                 <origin rpy="0 0 0" xyz="0 0 0" />
                 <geometry>
-                    <mesh filename="file://$(find gen3_lite_description)/meshes/upper_wrist_link.STL" />
-                </geometry>
-                <material name="">
-                    <color rgba="0.803 0.824 0.820 1" />
-                </material>
-            </visual>
-            <collision>
-                <origin rpy="0 0 0" xyz="0 0 0" />
-                <geometry>
-                    <mesh filename="file://$(find gen3_lite_description)/meshes/upper_wrist_link.STL" />
+                    <mesh filename="package://gen3_lite_description/meshes/upper_wrist_link.STL" />
+                </geometry>
+                <material name="">
+                    <color rgba="0.803 0.824 0.820 1" />
+                </material>
+            </visual>
+            <collision>
+                <origin rpy="0 0 0" xyz="0 0 0" />
+                <geometry>
+                    <mesh filename="package://gen3_lite_description/meshes/upper_wrist_link.STL" />
                 </geometry>
             </collision>

File: grippers/kinova_2f_lite/kinova_2f_lite_description/urdf/kinova_2f_lite_macro.urdf.xacro (robot description, xacro)
@@ -35,5 +35,5 @@
                 <origin rpy="0 0 0" xyz="0 0 0" />
                 <geometry>
-                    <mesh filename="file://$(find kinova_2f_lite_description)/meshes/gripper_base_link.STL" />
+                    <mesh filename="package://kinova_2f_lite_description/meshes/gripper_base_link.STL" />
                 </geometry>
                 <material name="">
@@ -44,5 +44,5 @@
                 <origin rpy="0 0 0" xyz="0 0 0" />
                 <geometry>
-                    <mesh filename="file://$(find kinova_2f_lite_description)/meshes/gripper_base_link.STL" />
+                    <mesh filename="package://kinova_2f_lite_description/meshes/gripper_base_link.STL" />
                 </geometry>
             </collision>
@@ -60,5 +60,5 @@
                 <origin rpy="0 0 0" xyz="0 0 0" />
                 <geometry>
-                    <mesh filename="file://$(find kinova_2f_lite_description)/meshes/right_finger_prox_link.STL" />
+                    <mesh filename="package://kinova_2f_lite_description/meshes/right_finger_prox_link.STL" />
                 </geometry>
                 <material name="">
@@ -69,5 +69,5 @@
                 <origin rpy="0 0 0" xyz="0 0 0" />
                 <geometry>
-                    <mesh filename="file://$(find kinova_2f_lite_description)/meshes/right_finger_prox_link.STL" />
+                    <mesh filename="package://kinova_2f_lite_description/meshes/right_finger_prox_link.STL" />
                 </geometry>
             </collision>
@@ -94,5 +94,5 @@
                 <origin rpy="0 0 0" xyz="0 0 0" />
                 <geometry>
-                    <mesh filename="file://$(find kinova_2f_lite_description)/meshes/right_finger_dist_link.STL" />
+                    <mesh filename="package://kinova_2f_lite_description/meshes/right_finger_dist_link.STL" />
                 </geometry>
                 <material name="">
@@ -103,5 +103,5 @@
                 <origin rpy="0 0 0" xyz="0 0 0" />
                 <geometry>
-                    <mesh filename="file://$(find kinova_2f_lite_description)/meshes/right_finger_dist_link.STL" />
+                    <mesh filename="package://kinova_2f_lite_description/meshes/right_finger_dist_link.STL" />
                 </geometry>
             </collision>
@@ -129,5 +129,5 @@
                 <origin rpy="0 0 0" xyz="0 0 0" />
                 <geometry>
-                    <mesh filename="file://$(find kinova_2f_lite_description)/meshes/left_finger_prox_link.STL" />
+                    <mesh filename="package://kinova_2f_lite_description/meshes/left_finger_prox_link.STL" />
                 </geometry>
                 <material name="">
@@ -138,5 +138,5 @@
                 <origin rpy="0 0 0" xyz="0 0 0" />
                 <geometry>
-                    <mesh filename="file://$(find kinova_2f_lite_description)/meshes/left_finger_prox_link.STL" />
+                    <mesh filename="package://kinova_2f_lite_description/meshes/left_finger_prox_link.STL" />
                 </geometry>
             </collision>
@@ -164,5 +164,5 @@
                 <origin rpy="0 0 0" xyz="0 0 0" />
                 <geometry>
-                    <mesh filename="file://$(find kinova_2f_lite_description)/meshes/left_finger_dist_link.STL" />
+                    <mesh filename="package://kinova_2f_lite_description/meshes/left_finger_dist_link.STL" />
                 </geometry>
                 <material name="">
@@ -173,5 +173,5 @@
                 <origin rpy="0 0 0" xyz="0 0 0" />
                 <geometry>
-                    <mesh filename="file://$(find kinova_2f_lite_description)/meshes/left_finger_dist_link.STL" />
+                    <mesh filename="package://kinova_2f_lite_description/meshes/left_finger_dist_link.STL" />
                 </geometry>
             </collision>
