Commit message: fix ros2 control problems

File: gen3_lite/gen3_lite_description/urdf/gen3_lite_macro.urdf.xacro (robot description, xacro)
@@ -218,5 +218,5 @@
         <xacro:if value="${sim_gazebo}">
             <xacro:include filename="$(find gen3_lite_description)/urdf/gz/gen3_lite.gazebo.xacro" />
-            <xacro:gen3_lite_gazebo prefix="${prefix}" use_camera="${use_camera}" />
+            <xacro:gen3_lite_gazebo parent="${parent}" prefix="${prefix}" use_camera="${use_camera}" />
         </xacro:if>
         <xacro:include filename="$(find gen3_lite_description)/urdf/ros2_control/gen3_lite_ros2_control.xacro" />

File: gen3_lite/gen3_lite_description/urdf/gz/gen3_lite.gazebo.xacro (robot description, xacro)
@@ -1,5 +1,5 @@
 <?xml version="1.0"?>
 <robot xmlns:xacro="http://ros.org/wiki/xacro">
-  <xacro:macro name="gen3_lite_gazebo" params="prefix use_camera">
+  <xacro:macro name="gen3_lite_gazebo" params="parent prefix use_camera">
     <gazebo reference="${prefix}base_link">
         <material>Kortex/Gray</material>
@@ -43,12 +43,15 @@
     </xacro:if>
     <!-- ROS2 CONTROL -->
-    <gazebo>
-      <plugin filename="gz_ros2_control-system" name="gz_ros2_control::GazeboSimROS2ControlPlugin">
-        <ros>
-          <namespace>$(arg namespace)</namespace>
-        </ros>
-        <parameters>$(find arms_bringup)/config/ros2_control.yaml</parameters>
-      </plugin>
-    </gazebo>
+    <!-- condition to avoid conflicts when launching the arm as an accessory. -->
+    <xacro:if value="${parent == 'world'}">
+      <gazebo>
+        <plugin filename="gz_ros2_control-system" name="gz_ros2_control::GazeboSimROS2ControlPlugin">
+          <ros>
+            <namespace>$(arg namespace)</namespace>
+          </ros>
+          <parameters>$(find arms_bringup)/config/ros2_control.yaml</parameters>
+        </plugin>
+      </gazebo>
+    </xacro:if>
   </xacro:macro>
 </robot>

Commit message: add a camera attached to the end_effector link

File: gen3_lite/gen3_lite_description/urdf/gen3_lite_macro.urdf.xacro (robot description, xacro)
@@ -1,14 +1,8 @@
 <?xml version="1.0"?>
 <robot xmlns:xacro="http://ros.org/wiki/xacro">
+    <xacro:include filename="$(find gen3_lite_description)/urdf/macros.urdf.xacro" />
     <!-- Propagate last link name information because it is the gripper's parent link -->
     <xacro:property name="last_arm_link" value="dummy_link"/>
-    <xacro:include filename="$(find gen3_lite_description)/urdf/macros.urdf.xacro" />
-    <xacro:macro name="load_arm" params="
-        *origin
-        parent
-        prefix
-        sim_gazebo
-        gripper
-        use_camera">
+    <xacro:macro name="load_arm" params="*origin parent prefix sim_gazebo gripper use_camera">
         <joint name="${prefix}base_joint" type="fixed">
             <xacro:insert_block name="origin" />
@@ -30,7 +24,5 @@
                     <mesh filename="package://gen3_lite_description/meshes/base_link.STL" />
                 </geometry>
-                <material name="">
-                    <color rgba="0.803 0.824 0.820 1" />
-                </material>
+                <material name="gen3_lite_white" />
             </visual>
             <collision>
@@ -55,7 +47,5 @@
                     <mesh filename="package://gen3_lite_description/meshes/shoulder_link.STL" />
                 </geometry>
-                <material name="">
-                    <color rgba="0.803 0.824 0.820 1" />
-                </material>
+                <material name="gen3_lite_white" />
             </visual>
             <collision>
@@ -73,5 +63,4 @@
             <limit lower="${min_joint_1_pos}" upper="${max_joint_1_pos}"
                     effort="${joint_1_effort}" velocity="${joint_1_vel}" />
-            <!-- <dynamics damping="2.0" friction="0.2"/> -->
         </joint>
         <link name="${prefix}arm_link">
@@ -89,7 +78,5 @@
                     <mesh filename="package://gen3_lite_description/meshes/arm_link.STL" />
                 </geometry>
-                <material name="">
-                    <color rgba="0.803 0.824 0.820 1" />
-                </material>
+                <material name="gen3_lite_white" />
             </visual>
             <collision>
@@ -107,5 +94,4 @@
             <limit lower="${min_joint_2_pos}" upper="${max_joint_2_pos}"
                     effort="${joint_2_effort}" velocity="${joint_2_vel}" />
-            <!-- <dynamics damping="3.0" friction="0.3"/> -->
         </joint>
         <link name="${prefix}forearm_link">
@@ -123,7 +109,5 @@
                     <mesh filename="package://gen3_lite_description/meshes/forearm_link.STL" />
                 </geometry>
-                <material name="">
-                    <color rgba="0.803 0.824 0.820 1" />
-                </material>
+                <material name="gen3_lite_white" />
             </visual>
             <collision>
@@ -141,5 +125,4 @@
             <limit lower="${min_joint_3_pos}" upper="${max_joint_3_pos}"
                     effort="${joint_3_effort}" velocity="${joint_3_vel}" />
-            <!-- <dynamics damping="2.5" friction="0.25"/> -->
         </joint>
         <link name="${prefix}lower_wrist_link">
@@ -157,7 +140,5 @@
                     <mesh filename="package://gen3_lite_description/meshes/lower_wrist_link.STL" />
                 </geometry>
-                <material name="">
-                    <color rgba="0.803 0.824 0.820 1" />
-                </material>
+                <material name="gen3_lite_white" />
             </visual>
             <collision>
@@ -175,5 +156,4 @@
             <limit lower="${min_joint_4_pos}" upper="${max_joint_4_pos}"
                     effort="${joint_4_effort}" velocity="${joint_4_vel}" />
-            <!-- <dynamics damping="1.0" friction="0.1"/> -->
         </joint>
         <link name="${prefix}upper_wrist_link">
@@ -191,7 +171,5 @@
                     <mesh filename="package://gen3_lite_description/meshes/upper_wrist_link.STL" />
                 </geometry>
-                <material name="">
-                    <color rgba="0.803 0.824 0.820 1" />
-                </material>
+                <material name="gen3_lite_white" />
             </visual>
             <collision>
@@ -209,5 +187,4 @@
             <limit lower="${min_joint_5_pos}" upper="${max_joint_5_pos}"
                     effort="${joint_5_effort}" velocity="${joint_5_vel}" />
-            <!-- <dynamics damping="1.0" friction="0.1"/> -->
         </joint>
         <link name="${prefix}end_effector_link">
@@ -228,6 +205,6 @@
             <limit lower="${min_joint_6_pos}" upper="${max_joint_6_pos}"
                     effort="${joint_6_effort}" velocity="${joint_6_vel}" />
-            <!-- <dynamics damping="1.0" friction="0.1"/> -->
-        </joint>
+        </joint>
+        <!-- Dummy Link for Gripper Attachment -->
         <link name="${prefix}dummy_link" />
         <joint name="${prefix}end_effector" type="fixed">
@@ -236,11 +213,15 @@
             <child link="${prefix}dummy_link" />
             <axis xyz="0 0 1" />
-            <!-- <limit lower="0" upper="0" effort="0" velocity="0" /> -->
-        </joint>
+        </joint>
+        <!-- Optional components -->
         <xacro:if value="${use_camera}">
-            <xacro:include filename="$(find gen3_lite_description)/urdf/camera/d435.urdf.xacro" />
+            <!-- <xacro:include filename="$(find gen3_lite_description)/urdf/camera/d435.urdf.xacro" />
             <xacro:d435_camera parent="base_link" prefix="${prefix}">
                 <origin rpy="0 0 0" xyz="0.22 -0.30 0" />
-            </xacro:d435_camera>
+            </xacro:d435_camera> -->
+            <xacro:include filename="$(find gen3_lite_description)/urdf/camera/_d435.urdf.xacro" />
+            <xacro:sensor_d435 parent="dummy_link" prefix="${prefix}" name="camera_1">
+                <origin rpy="${M_PI} -${M_PI/2} 0.0" xyz="0.045 0.0 0.015" />
+            </xacro:sensor_d435>
         </xacro:if>
         <xacro:if value="${sim_gazebo}">

File: gen3_lite/gen3_lite_description/urdf/gz/gen3_lite.gazebo.xacro (robot description, xacro)
@@ -21,6 +21,6 @@
         </gazebo>
         <xacro:if value="${use_camera}">
-        <gazebo reference="${prefix}camera_head_link">
-            <sensor name="${prefix}camera_head" type="rgbd_camera">
+        <gazebo reference="${prefix}camera_1_link">
+            <sensor name="${prefix}camera_1" type="rgbd_camera">
                 <camera>
                     <horizontal_fov>1.5184</horizontal_fov>
@@ -35,6 +35,6 @@
                 </camera>
                 <always_on>1</always_on>
-                <gz_frame_id>${prefix}camera_head_link</gz_frame_id>
-                <topic>${prefix}camera_head</topic>
+                <gz_frame_id>${prefix}camera_1_link</gz_frame_id>
+                <topic>${prefix}camera_1</topic>
                 <update_rate>5</update_rate>
                 <visualize>true</visualize>
