Commit message: improve readability

File: gen3_lite/gen3_lite_description/urdf/gen3_lite.urdf.xacro (robot description, xacro)
@@ -1,4 +1,4 @@
 <?xml version="1.0"?>
-<robot name="$(arg name)" xmlns:xacro="http://ros.org/wiki/xacro">
+<robot name="gen3_lite" xmlns:xacro="http://ros.org/wiki/xacro">
     <!-- Arguments -->
     <xacro:arg name="sim_gazebo" default="false" />
@@ -6,28 +6,12 @@
     <xacro:arg name="prefix" default=""/>
     <xacro:arg name="gripper" default="" />
-    <xacro:arg name="joint_limits" default="$(find gen3_lite_description)/config/joint_limits.yaml" />
-    <xacro:arg name="initial_position" default="$(find gen3_lite_description)/config/initial_position.yaml" />
-    <!-- Not used yet -->
-    <xacro:arg name="vision" default="false" />
-    <xacro:arg name="robot_ip" default="192.168.1.10" />
-    <xacro:arg name="username" default="admin" />
-    <xacro:arg name="password" default="admin" />
-    <xacro:arg name="port" default="10000" />
-    <xacro:arg name="port_realtime" default="10001" />
-    <xacro:arg name="session_inactivity_timeout_ms" default="60000" />
-    <xacro:arg name="connection_inactivity_timeout_ms" default="2000" />
-    <xacro:arg name="gripper_joint_name" default="right_finger_bottom_joint" />
-    <xacro:arg name="gripper_max_velocity" default="100.0" />
-    <xacro:arg name="gripper_max_force" default="100.0" />
-    <xacro:arg name="use_internal_bus_gripper_comm" default="true" />
-    <xacro:arg name="use_external_cable" default="false" />
     <xacro:include filename="$(find gen3_lite_description)/urdf/gen3_lite_macro.urdf.xacro" />
     <link name="world"/>
     <xacro:load_arm
-        parent="world"
-        prefix="$(arg prefix)"
-        sim_gazebo="$(arg sim_gazebo)"
-        gripper="$(arg gripper)"
-        use_camera="$(arg use_camera)">
+            parent="world"
+            prefix="$(arg prefix)"
+            sim_gazebo="$(arg sim_gazebo)"
+            gripper="$(arg gripper)"
+            use_camera="$(arg use_camera)">
         <origin rpy="0 0 0" xyz="0 0 0" />
     </xacro:load_arm>

File: gen3_lite/gen3_lite_description/urdf/macros.urdf.xacro (robot description, xacro)
@@ -1,39 +1,48 @@
 <?xml version="1.0"?>
 <robot xmlns:xacro="http://ros.org/wiki/xacro">
+    <xacro:property name="M_PI" value="3.1415926535897931" />
+    <xacro:arg name="joint_limits" default="$(find gen3_lite_description)/config/joint_limits.yaml" />
+    <xacro:arg name="initial_position" default="$(find gen3_lite_description)/config/initial_position.yaml" />
+    <xacro:arg name="hardware" default="$(find gen3_lite_description)/config/hardware.yaml" />
+    <material name="gen3_lite_white">
+        <color rgba="0.803 0.824 0.820 1" />
+    </material>
     <xacro:property name="joint_limits_config" value="${xacro.load_yaml('$(arg joint_limits)')}" />
     <xacro:property name="initial_positions_config" value="${xacro.load_yaml('$(arg initial_position)')}" />
+    <xacro:property name="hardware_config" value="${xacro.load_yaml('$(arg hardware)')}" />
+    <xacro:macro name="load_joint_limits" params="joint">
     <!-- Position limits -->
-    <xacro:property name="min_joint_1_pos" value="${joint_limits_config['joint_limits']['joint_1']['min_position']}" />
-    <xacro:property name="max_joint_1_pos" value="${joint_limits_config['joint_limits']['joint_1']['max_position']}" />
-    <xacro:property name="min_joint_2_pos" value="${joint_limits_config['joint_limits']['joint_2']['min_position']}" />
-    <xacro:property name="max_joint_2_pos" value="${joint_limits_config['joint_limits']['joint_2']['max_position']}" />
-    <xacro:property name="min_joint_3_pos" value="${joint_limits_config['joint_limits']['joint_3']['min_position']}" />
-    <xacro:property name="max_joint_3_pos" value="${joint_limits_config['joint_limits']['joint_3']['max_position']}" />
-    <xacro:property name="min_joint_4_pos" value="${joint_limits_config['joint_limits']['joint_4']['min_position']}" />
-    <xacro:property name="max_joint_4_pos" value="${joint_limits_config['joint_limits']['joint_4']['max_position']}" />
-    <xacro:property name="min_joint_5_pos" value="${joint_limits_config['joint_limits']['joint_5']['min_position']}" />
-    <xacro:property name="max_joint_5_pos" value="${joint_limits_config['joint_limits']['joint_5']['max_position']}" />
-    <xacro:property name="min_joint_6_pos" value="${joint_limits_config['joint_limits']['joint_6']['min_position']}" />
-    <xacro:property name="max_joint_6_pos" value="${joint_limits_config['joint_limits']['joint_6']['max_position']}" />
+        <xacro:property name="min_${joint}_pos"
+            value="${joint_limits_config['joint_limits'][joint]['min_position']}" scope="parent" />
+        <xacro:property name="max_${joint}_pos"
+            value="${joint_limits_config['joint_limits'][joint]['max_position']}" scope="parent" />
     <!-- Velocity limits -->
-    <xacro:property name="joint_1_vel" value="${joint_limits_config['joint_limits']['joint_1']['max_velocity']}" />
-    <xacro:property name="joint_2_vel" value="${joint_limits_config['joint_limits']['joint_2']['max_velocity']}" />
-    <xacro:property name="joint_3_vel" value="${joint_limits_config['joint_limits']['joint_3']['max_velocity']}" />
-    <xacro:property name="joint_4_vel" value="${joint_limits_config['joint_limits']['joint_4']['max_velocity']}" />
-    <xacro:property name="joint_5_vel" value="${joint_limits_config['joint_limits']['joint_5']['max_velocity']}" />
-    <xacro:property name="joint_6_vel" value="${joint_limits_config['joint_limits']['joint_6']['max_velocity']}" />
+        <xacro:property name="${joint}_vel"
+            value="${joint_limits_config['joint_limits'][joint]['max_velocity']}" scope="parent" />
     <!-- Effort limits -->
-    <xacro:property name="joint_1_effort" value="${joint_limits_config['joint_limits']['joint_1']['max_effort']}" />
-    <xacro:property name="joint_2_effort" value="${joint_limits_config['joint_limits']['joint_2']['max_effort']}" />
-    <xacro:property name="joint_3_effort" value="${joint_limits_config['joint_limits']['joint_3']['max_effort']}" />
-    <xacro:property name="joint_4_effort" value="${joint_limits_config['joint_limits']['joint_4']['max_effort']}" />
-    <xacro:property name="joint_5_effort" value="${joint_limits_config['joint_limits']['joint_5']['max_effort']}" />
-    <xacro:property name="joint_6_effort" value="${joint_limits_config['joint_limits']['joint_6']['max_effort']}" />
+        <xacro:property name="${joint}_effort"
+            value="${joint_limits_config['joint_limits'][joint]['max_effort']}" scope="parent" />
     <!-- Access initial positions -->
-    <xacro:property name="joint_1_initial" value="${initial_positions_config['initial_positions']['joint_1']}" />
-    <xacro:property name="joint_2_initial" value="${initial_positions_config['initial_positions']['joint_2']}" />
-    <xacro:property name="joint_3_initial" value="${initial_positions_config['initial_positions']['joint_3']}" />
-    <xacro:property name="joint_4_initial" value="${initial_positions_config['initial_positions']['joint_4']}" />
-    <xacro:property name="joint_5_initial" value="${initial_positions_config['initial_positions']['joint_5']}" />
-    <xacro:property name="joint_6_initial" value="${initial_positions_config['initial_positions']['joint_6']}" />
+        <xacro:property name="${joint}_initial"
+            value="${initial_positions_config['initial_positions'][joint]}" scope="parent" />
+    </xacro:macro>
+    <!-- Load properties for all 6 joints -->
+    <xacro:load_joint_limits joint="joint_1" />
+    <xacro:load_joint_limits joint="joint_2" />
+    <xacro:load_joint_limits joint="joint_3" />
+    <xacro:load_joint_limits joint="joint_4" />
+    <xacro:load_joint_limits joint="joint_5" />
+    <xacro:load_joint_limits joint="joint_6" />
+    <!-- Hardware Configuration -->
+    <xacro:property name="robot_ip" value="${hardware_config['hardware']['robot_ip']}" />
+    <xacro:property name="username" value="${hardware_config['hardware']['username']}" />
+    <xacro:property name="password" value="${hardware_config['hardware']['password']}" />
+    <xacro:property name="port" value="${hardware_config['hardware']['port']}" />
+    <xacro:property name="port_realtime" value="${hardware_config['hardware']['port_realtime']}" />
+    <xacro:property name="session_inactivity_timeout_ms" value="${hardware_config['hardware']['session_inactivity_timeout_ms']}" />
+    <xacro:property name="connection_inactivity_timeout_ms" value="${hardware_config['hardware']['connection_inactivity_timeout_ms']}" />
+    <xacro:property name="use_internal_bus_gripper_comm" value="${hardware_config['hardware']['use_internal_bus_gripper_comm']}" />
+    <xacro:property name="gripper_joint_name" value="${hardware_config['hardware']['gripper_joint_name']}" />
+    <xacro:property name="gripper_max_velocity" value="${hardware_config['hardware']['gripper_max_velocity']}" />
+    <xacro:property name="gripper_max_force" value="${hardware_config['hardware']['gripper_max_force']}" />
 </robot>
