Commit message: add robot description

File: unitree_d1/unitree_d1_description/urdf/gz/unitree_d1.gazebo.xacro (robot description, xacro)
@@ -24,24 +24,24 @@
     </gazebo>
     <xacro:if value="${use_camera}">
-      <gazebo reference="${prefix}camera_head_link">
-        <sensor name="${prefix}camera_head" type="rgbd_camera">
-          <camera>
-            <horizontal_fov>1.5184</horizontal_fov>
-            <image>
-              <width>424</width>
-              <height>240</height>
-            </image>
-            <clip>
-              <near>0.05</near>
-              <far>1.5</far>
-            </clip>
-          </camera>
-          <always_on>1</always_on>
-          <gz_frame_id>${prefix}camera_head_link</gz_frame_id>
-          <topic>${prefix}camera_head</topic>
-          <update_rate>5</update_rate>
-          <visualize>true</visualize>
-        </sensor>
-      </gazebo>
+        <gazebo reference="${prefix}camera_1_link">
+            <sensor name="${prefix}camera_1" type="rgbd_camera">
+                <camera>
+                    <horizontal_fov>1.5184</horizontal_fov>
+                    <image>
+                        <width>640</width>
+                        <height>480</height>
+                    </image>
+                    <clip>
+                        <near>0.05</near>
+                        <far>1.5</far>
+                    </clip>
+                </camera>
+                <always_on>1</always_on>
+                <gz_frame_id>${prefix}camera_1_link</gz_frame_id>
+                <topic>${prefix}camera_1</topic>
+                <update_rate>5</update_rate>
+                <visualize>true</visualize>
+            </sensor>
+        </gazebo>
     </xacro:if>
     <!-- ROS2 CONTROL -->

File: unitree_d1/unitree_d1_description/urdf/macros.urdf.xacro (robot description, xacro)
@@ -1,49 +1,37 @@
 <?xml version="1.0"?>
 <robot xmlns:xacro="http://ros.org/wiki/xacro">
+    <xacro:property name="M_PI" value="3.1415926535897931" />
+    <xacro:arg name="joint_limits" default="$(find unitree_d1_description)/config/joint_limits.yaml" />
+    <xacro:arg name="initial_position" default="$(find unitree_d1_description)/config/initial_position.yaml" />
     <xacro:property name="joint_limits_config" value="${xacro.load_yaml('$(arg joint_limits)')}" />
     <xacro:property name="initial_positions_config" value="${xacro.load_yaml('$(arg initial_position)')}" />
+    <xacro:macro name="load_joint_limits" params="joint">
     <!-- Position limits -->
-    <xacro:property name="min_joint_1_pos" value="${joint_limits_config['joint_limits']['joint_1']['min_position']}" />
-    <xacro:property name="max_joint_1_pos" value="${joint_limits_config['joint_limits']['joint_1']['max_position']}" />
-    <xacro:property name="min_joint_2_pos" value="${joint_limits_config['joint_limits']['joint_2']['min_position']}" />
-    <xacro:property name="max_joint_2_pos" value="${joint_limits_config['joint_limits']['joint_2']['max_position']}" />
-    <xacro:property name="min_joint_3_pos" value="${joint_limits_config['joint_limits']['joint_3']['min_position']}" />
-    <xacro:property name="max_joint_3_pos" value="${joint_limits_config['joint_limits']['joint_3']['max_position']}" />
-    <xacro:property name="min_joint_4_pos" value="${joint_limits_config['joint_limits']['joint_4']['min_position']}" />
-    <xacro:property name="max_joint_4_pos" value="${joint_limits_config['joint_limits']['joint_4']['max_position']}" />
-    <xacro:property name="min_joint_5_pos" value="${joint_limits_config['joint_limits']['joint_5']['min_position']}" />
-    <xacro:property name="max_joint_5_pos" value="${joint_limits_config['joint_limits']['joint_5']['max_position']}" />
-    <xacro:property name="min_joint_6_pos" value="${joint_limits_config['joint_limits']['joint_6']['min_position']}" />
-    <xacro:property name="max_joint_6_pos" value="${joint_limits_config['joint_limits']['joint_6']['max_position']}" />
+        <xacro:property name="min_${joint}_pos"
+            value="${joint_limits_config['joint_limits'][joint]['min_position']}" scope="parent" />
+        <xacro:property name="max_${joint}_pos"
+            value="${joint_limits_config['joint_limits'][joint]['max_position']}" scope="parent" />
     <!-- Velocity limits -->
-    <xacro:property name="joint_1_vel" value="${joint_limits_config['joint_limits']['joint_1']['max_velocity']}" />
-    <xacro:property name="joint_2_vel" value="${joint_limits_config['joint_limits']['joint_2']['max_velocity']}" />
-    <xacro:property name="joint_3_vel" value="${joint_limits_config['joint_limits']['joint_3']['max_velocity']}" />
-    <xacro:property name="joint_4_vel" value="${joint_limits_config['joint_limits']['joint_4']['max_velocity']}" />
-    <xacro:property name="joint_5_vel" value="${joint_limits_config['joint_limits']['joint_5']['max_velocity']}" />
-    <xacro:property name="joint_6_vel" value="${joint_limits_config['joint_limits']['joint_6']['max_velocity']}" />
+        <xacro:property name="${joint}_vel"
+            value="${joint_limits_config['joint_limits'][joint]['max_velocity']}" scope="parent" />
     <!-- Effort limits -->
-    <xacro:property name="joint_1_effort" value="${joint_limits_config['joint_limits']['joint_1']['max_effort']}" />
-    <xacro:property name="joint_2_effort" value="${joint_limits_config['joint_limits']['joint_2']['max_effort']}" />
-    <xacro:property name="joint_3_effort" value="${joint_limits_config['joint_limits']['joint_3']['max_effort']}" />
-    <xacro:property name="joint_4_effort" value="${joint_limits_config['joint_limits']['joint_4']['max_effort']}" />
-    <xacro:property name="joint_5_effort" value="${joint_limits_config['joint_limits']['joint_5']['max_effort']}" />
-    <xacro:property name="joint_6_effort" value="${joint_limits_config['joint_limits']['joint_6']['max_effort']}" />
+        <xacro:property name="${joint}_effort"
+            value="${joint_limits_config['joint_limits'][joint]['max_effort']}" scope="parent" />
     <!-- Access initial positions -->
-    <xacro:property name="joint_1_initial" value="${initial_positions_config['initial_positions']['joint_1']}" />
-    <xacro:property name="joint_2_initial" value="${initial_positions_config['initial_positions']['joint_2']}" />
-    <xacro:property name="joint_3_initial" value="${initial_positions_config['initial_positions']['joint_3']}" />
-    <xacro:property name="joint_4_initial" value="${initial_positions_config['initial_positions']['joint_4']}" />
-    <xacro:property name="joint_5_initial" value="${initial_positions_config['initial_positions']['joint_5']}" />
-    <xacro:property name="joint_6_initial" value="${initial_positions_config['initial_positions']['joint_6']}" />
-    <xacro:property name="material_black">
-        <material name="black">
-            <color rgba="0.1 0.1 0.1 1"/>
-        </material>
-    </xacro:property>
-    <xacro:property name="material_dark_grey">
-        <material name="dark_grey">
-            <color rgba="0.3 0.3 0.3 1"/>
-        </material>
-    </xacro:property>
+        <xacro:property name="${joint}_initial"
+            value="${initial_positions_config['initial_positions'][joint]}" scope="parent" />
+    </xacro:macro>
+    <!-- Load properties for all 6 joints -->
+    <xacro:load_joint_limits joint="joint_1" />
+    <xacro:load_joint_limits joint="joint_2" />
+    <xacro:load_joint_limits joint="joint_3" />
+    <xacro:load_joint_limits joint="joint_4" />
+    <xacro:load_joint_limits joint="joint_5" />
+    <xacro:load_joint_limits joint="joint_6" />
+    <material name="d1_black">
+        <color rgba="0.1 0.1 0.1 1"/>
+    </material>
+    <material name="d1_dark_grey">
+        <color rgba="0.25 0.25 0.25 1"/>
+    </material>
 </robot>

File: unitree_d1/unitree_d1_description/urdf/unitree_d1.urdf.xacro (robot description, xacro)
@@ -1,20 +1,19 @@
 <?xml version="1.0"?>
-<robot name="unitree_d1" xmlns:xacro="http://ros.org/wiki/xacro">
+<robot name="$(arg name)" xmlns:xacro="http://ros.org/wiki/xacro">
     <!-- Arguments -->
+    <xacro:arg name="name" default="unitree_d1" />
     <xacro:arg name="sim_gazebo" default="true" />
     <xacro:arg name="use_camera" default="false" />
     <xacro:arg name="prefix" default=""/>
     <xacro:arg name="gripper" default="" />
-    <xacro:arg name="joint_limits" default="$(find unitree_d1_description)/config/joint_limits.yaml" />
-    <xacro:arg name="initial_position" default="$(find unitree_d1_description)/config/initial_position.yaml" />
+    <xacro:include filename="$(find unitree_d1_description)/urdf/camera/_materials.urdf.xacro" />
     <xacro:include filename="$(find unitree_d1_description)/urdf/unitree_d1_macro.urdf.xacro" />
-    <xacro:include filename="$(find unitree_d1_description)/urdf/macros.urdf.xacro" />
     <link name="world"/>
     <xacro:load_arm
-        parent="world"
-        prefix="$(arg prefix)"
-        sim_gazebo="$(arg sim_gazebo)"
-        gripper="$(arg gripper)"
-        use_camera="$(arg use_camera)">
+            parent="world"
+            prefix="$(arg prefix)"
+            sim_gazebo="$(arg sim_gazebo)"
+            gripper="$(arg gripper)"
+            use_camera="$(arg use_camera)">
         <origin rpy="0 0 0" xyz="0 0 0" />
     </xacro:load_arm>

File: unitree_d1/unitree_d1_description/urdf/unitree_d1_macro.urdf.xacro (robot description, xacro)
@@ -1,10 +1,11 @@
 <?xml version="1.0"?>
 <robot xmlns:xacro="http://ros.org/wiki/xacro">
+    <xacro:include filename="$(find unitree_d1_description)/urdf/macros.urdf.xacro" />
     <!-- Propagate last link name information because it is the gripper's parent link -->
-    <xacro:property name="last_arm_link" value="Link6"/>
+    <xacro:property name="last_arm_link" value="Link6" />
     <xacro:macro name="load_arm" params="*origin parent prefix sim_gazebo gripper use_camera">
         <joint name="${prefix}base_joint" type="fixed">
             <xacro:insert_block name="origin" />
-            <parent link="${parent}"/>
+            <parent link="${parent}" />
             <child link="${prefix}base_link" />
         </joint>
@@ -21,12 +22,12 @@
                 <origin rpy="0 0 0" xyz="0 0 0" />
                 <geometry>
-                    <mesh filename="file://$(find unitree_d1_description)/meshes/base_link.STL" />
-                </geometry>
-                <xacro:insert_block name="material_black" />
-            </visual>
-            <collision>
-                <origin rpy="0 0 0" xyz="0 0 0" />
-                <geometry>
-                    <mesh filename="file://$(find unitree_d1_description)/meshes/base_link.STL" />
+                    <mesh filename="package://unitree_d1_description/meshes/base_link.STL" />
+                </geometry>
+                <material name="d1_dark_grey" />
+            </visual>
+            <collision>
+                <origin rpy="0 0 0" xyz="0 0 0" />
+                <geometry>
+                    <mesh filename="package://unitree_d1_description/meshes/base_link.STL" />
                 </geometry>
             </collision>
@@ -44,12 +45,12 @@
                 <origin rpy="0 0 0" xyz="0 0 0" />
                 <geometry>
-                    <mesh filename="file://$(find unitree_d1_description)/meshes/Link1.STL" />
-                </geometry>
-                <xacro:insert_block name="material_black" />
+                    <mesh filename="package://unitree_d1_description/meshes/Link1.STL" />
+                </geometry>
+                <material name="d1_dark_grey" />
             </visual>
             <collision>
                 <origin xyz="0 0 0" rpy="0 0 0" />
                 <geometry>
-                    <mesh filename="file://$(find unitree_d1_description)/meshes/Link1.STL" />
+                    <mesh filename="package://unitree_d1_description/meshes/Link1.STL" />
                 </geometry>
             </collision>
@@ -75,12 +76,12 @@
                 <origin rpy="0 0 0" xyz="0 0 0" />
                 <geometry>
-                    <mesh filename="file://$(find unitree_d1_description)/meshes/Link2.STL"/>
-                </geometry>
-                <xacro:insert_block name="material_black"/>
-            </visual>
-            <collision>
-                <origin rpy="0 0 0" xyz="0 0 0" />
-                <geometry>
-                    <mesh filename="file://$(find unitree_d1_description)/meshes/Link2.STL"/>
+                    <mesh filename="package://unitree_d1_description/meshes/Link2.STL" />
+                </geometry>
+                <material name="d1_dark_grey" />
+            </visual>
+            <collision>
+                <origin rpy="0 0 0" xyz="0 0 0" />
+                <geometry>
+                    <mesh filename="package://unitree_d1_description/meshes/Link2.STL" />
                 </geometry>
             </collision>
@@ -106,12 +107,12 @@
                 <origin rpy="0 0 0" xyz="0 0 0" />
                 <geometry>
-                    <mesh filename="file://$(find unitree_d1_description)/meshes/Link3.STL" />
-                </geometry>
-                <xacro:insert_block name="material_black" />
-            </visual>
-            <collision>
-                <origin rpy="0 0 0" xyz="0 0 0" />
-                <geometry>
-                    <mesh filename="file://$(find unitree_d1_description)/meshes/Link3.STL" />
+                    <mesh filename="package://unitree_d1_description/meshes/Link3.STL" />
+                </geometry>
+                <material name="d1_dark_grey" />
+            </visual>
+            <collision>
+                <origin rpy="0 0 0" xyz="0 0 0" />
+                <geometry>
+                    <mesh filename="package://unitree_d1_description/meshes/Link3.STL" />
                 </geometry>
             </collision>
@@ -137,12 +138,12 @@
                 <origin rpy="0 0 0" xyz="0 0 0" />
                 <geometry>
-                    <mesh filename="file://$(find unitree_d1_description)/meshes/Link4.STL" />
-                </geometry>
-                <xacro:insert_block name="material_black" />
-            </visual>
-            <collision>
-                <origin rpy="0 0 0" xyz="0 0 0" />
-                <geometry>
-                    <mesh filename="file://$(find unitree_d1_description)/meshes/Link4.STL" />
+                    <mesh filename="package://unitree_d1_description/meshes/Link4.STL" />
+                </geometry>
+                <material name="d1_dark_grey" />
+            </visual>
+            <collision>
+                <origin rpy="0 0 0" xyz="0 0 0" />
+                <geometry>
+                    <mesh filename="package://unitree_d1_description/meshes/Link4.STL" />
                 </geometry>
             </collision>
@@ -150,7 +151,7 @@
         <joint name="${prefix}joint_4" type="revolute">
             <origin rpy="-1.5708 0 -1.5708" xyz="0.0577 0.042 -0.0275" />
-            <parent link="${prefix}Link3"/>
-            <child link="${prefix}Link4"/>
-            <axis xyz="0 0 1"/>
+            <parent link="${prefix}Link3" />
+            <child link="${prefix}Link4" />
+            <axis xyz="0 0 1" />
             <limit lower="${min_joint_4_pos}" upper="${max_joint_4_pos}"
                     effort="${joint_4_effort}" velocity="${joint_4_vel}" />
@@ -168,12 +169,12 @@
                 <origin xyz="0 0 0" rpy="0 0 0" />
                 <geometry>
-                    <mesh filename="file://$(find unitree_d1_description)/meshes/Link5.STL" />
-                </geometry>
-                <xacro:insert_block name="material_black" />
-            </visual>
-            <collision>
-                <origin rpy="0 0 0" xyz="0 0 0" />
-                <geometry>
-                    <mesh filename="file://$(find unitree_d1_description)/meshes/Link5.STL" />
+                    <mesh filename="package://unitree_d1_description/meshes/Link5.STL" />
+                </geometry>
+                <material name="d1_dark_grey" />
+            </visual>
+            <collision>
+                <origin rpy="0 0 0" xyz="0 0 0" />
+                <geometry>
+                    <mesh filename="package://unitree_d1_description/meshes/Link5.STL" />
                 </geometry>
             </collision>
@@ -205,9 +206,10 @@
                     effort="${joint_6_effort}" velocity="${joint_6_vel}" />
         </joint>
+        <!-- Optional components -->
         <xacro:if value="${use_camera}">
-            <xacro:include filename="$(find unitree_d1_description)/urdf/camera/d435.urdf.xacro" />
-            <xacro:d435_camera parent="base_link" prefix="${prefix}">
-                <origin rpy="0 0 0" xyz="0.22 -0.60 0" />
-            </xacro:d435_camera>
+            <xacro:include filename="$(find unitree_d1_description)/urdf/camera/_d435.urdf.xacro" />
+            <xacro:sensor_d435 parent="${last_arm_link}" prefix="${prefix}" name="camera_1">
+                <origin rpy="0 -${M_PI/2} 0.0" xyz="-0.055 0.0 0.02" />
+            </xacro:sensor_d435>
         </xacro:if>
         <xacro:if value="${sim_gazebo}">
